File: hw/ShotClockProject/ShotClockProject.kicad_pcb (KiCad board)
At the start: 2 copper layers, 0 parts

Commit message: Init PCB
and start on broad layout phase
Parts:
- added BZ1: Buzzer, Buzzer_Beeper:Buzzer_CUI_CPT-9019S-SMT, F.Cu at (175.0, 66.8)
- added C1: 10u, Capacitor_SMD:C_0603_1608Metric, F.Cu at (159.2, 48.3)
- added C10: 10p, Capacitor_SMD:C_0603_1608Metric, F.Cu at (35.8, 49.8)
- added C11: 10p, Capacitor_SMD:C_0603_1608Metric, F.Cu at (35.8, 52.0)
- added C12: 1u, Capacitor_SMD:C_0603_1608Metric, F.Cu at (163.2, 58.4)
- added C13: 1u, Capacitor_SMD:C_0603_1608Metric, F.Cu at (163.2, 60.9)
- added C14: 10u, Capacitor_SMD:C_0603_1608Metric, F.Cu at (159.2, 91.3)
- added C15: 100n, Capacitor_SMD:C_0603_1608Metric, F.Cu at (159.2, 93.8)
- added C16: 10u, Capacitor_SMD:C_0603_1608Metric, F.Cu at (159.2, 96.3)
- added C17: 2.2p, Capacitor_SMD:C_0603_1608Metric, F.Cu at (179.5, 117.0)
- added C18: 10u, Capacitor_SMD:C_0603_1608Metric, F.Cu at (179.5, 119.6)
- added C19: 10u, Capacitor_SMD:C_0603_1608Metric, F.Cu at (179.5, 122.1)
- added C2: 100n, Capacitor_SMD:C_0603_1608Metric, F.Cu at (45.2, 43.2)
- added C20: 10u, Capacitor_SMD:C_0603_1608Metric, F.Cu at (179.5, 124.6)
- added C21: 0.1u, Capacitor_SMD:C_0603_1608Metric, F.Cu at (179.5, 127.1)
- added C22: 100n, Capacitor_SMD:C_0603_1608Metric, F.Cu at (159.2, 117.0)
- added C23: 100n, Capacitor_SMD:C_0603_1608Metric, F.Cu at (159.2, 119.6)
- added C24: 100n, Capacitor_SMD:C_0603_1608Metric, F.Cu at (159.2, 122.1)
- added C3: 100n, Capacitor_SMD:C_0603_1608Metric, F.Cu at (58.0, 47.5)
- added C4: 100n, Capacitor_SMD:C_0603_1608Metric, F.Cu at (45.8, 60.0)
- added C5: 100n, Capacitor_SMD:C_0603_1608Metric, F.Cu at (53.0, 60.0)
- added C6: 10n, Capacitor_SMD:C_0603_1608Metric, F.Cu at (40.8, 62.2)
- added C7: 1u, Capacitor_SMD:C_0603_1608Metric, F.Cu at (40.2, 54.0)
- added C8: 1u, Capacitor_SMD:C_0603_1608Metric, F.Cu at (42.0, 59.5)
- added C9: 100n, Capacitor_SMD:C_0603_1608Metric, F.Cu at (163.2, 50.8)
- added D1: Orange LED, LED_SMD:LED_0603_1608Metric, F.Cu at (191.2, 82.5)
- added D2: 1N4148, Diode_SMD:D_SOD-323, F.Cu at (189.6, 78.0)
- added D3: G_LED, LED_SMD:LED_0603_1608Metric, F.Cu at (167.8, 109.4)
- added D4: R_LED, LED_SMD:LED_0603_1608Metric, F.Cu at (167.8, 112.0)
- added FB1: 120R, Inductor_SMD:L_0603_1608Metric, F.Cu at (39.5, 59.5)
- added IC1: TP4056-42-ESOP8_Rearanged, Package_SO:Texas_HSOP-8-1EP_3.9x4.9mm_P1.27mm_ThermalVias, F.Cu at (161.5, 103.4)
- added J1: USB_C_Receptacle_USB2.0, Connector_USB:USB_C_Receptacle_Molex_105450-0101, F.Cu at (70.2, 50.9)
- added J10: Conn_01x33_Pin, Connector_PinHeader_2.54mm:PinHeader_1x33_P2.54mm_Horizontal, F.Cu at (144.1, 49.4)
- added J2: Conn_ST_STDC14, Connector_PinHeader_1.27mm:PinHeader_2x07_P1.27mm_Vertical_SMD, F.Cu at (188.5, 52.5)
- added J3: Conn_01x06_Pin, Connector_PinHeader_2.54mm:PinHeader_1x06_P2.54mm_Vertical_SMD_Pin1Left, F.Cu at (161.2, 73.3)
- added J4: Conn_01x03_Pin, Connector_PinHeader_1.00mm:PinHeader_1x03_P1.00mm_Vertical_SMD_Pin1Left, F.Cu at (168.5, 105.6)
- added J5: Conn_01x02_Pin, Connector_PinHeader_2.54mm:PinHeader_1x02_P2.54mm_Vertical_SMD_Pin1Left, F.Cu at (161.2, 110.2)
- added J6: Conn_01x03_Pin, Connector_PinHeader_2.54mm:PinHeader_1x03_P2.54mm_Vertical_SMD_Pin1Left, F.Cu at (173.2, 94.9)
- added J7: Conn_01x33_Pin, Connector_PinHeader_2.54mm:PinHeader_1x33_P2.54mm_Horizontal, F.Cu at (103.9, 49.4)
- added J8: Conn_01x33_Pin, Connector_PinHeader_2.54mm:PinHeader_1x33_P2.54mm_Horizontal, F.Cu at (117.3, 49.4)
- added J9: Conn_01x33_Pin, Connector_PinHeader_2.54mm:PinHeader_1x33_P2.54mm_Horizontal, F.Cu at (130.7, 49.4)
- added L1: L, Inductor_SMD:L_Sunlord_SWPA3012S, F.Cu at (183.8, 126.1)
- added NT1: NetTie_2, NetTie:NetTie-2_SMD_Pad2.0mm, F.Cu at (169.2, 101.6)
- added NT2: NetTie_2, NetTie:NetTie-2_SMD_Pad2.0mm, F.Cu at (185.0, 117.3)
- added Q1: Q_NPN_BCE, Package_TO_SOT_SMD:SOT-23, F.Cu at (181.5, 83.4)
- added Q2: Q_PMOS_SGD, Package_TO_SOT_SMD:SOT-23, F.Cu at (173.7, 105.3)
- added R1: 0R, Resistor_SMD:R_0603_1608Metric, F.Cu at (185.7, 98.2)
- added R10: 0.4R, Resistor_SMD:R_0603_1608Metric, F.Cu at (159.2, 98.8)
- added R11: 1k, Resistor_SMD:R_0603_1608Metric, F.Cu at (163.2, 91.3)
- added R12: 1M, Resistor_SMD:R_0603_1608Metric, F.Cu at (163.2, 93.8)
- added R13: 1k, Resistor_SMD:R_0603_1608Metric, F.Cu at (163.2, 96.3)
- added R14: 1k, Resistor_SMD:R_0603_1608Metric, F.Cu at (163.2, 98.8)
- added R15: 1M, Resistor_SMD:R_0603_1608Metric, F.Cu at (167.2, 91.3)
- added R16: 1k2, Resistor_SMD:R_0603_1608Metric, F.Cu at (167.2, 93.8)
- added R17: 4780R, Resistor_SMD:R_0603_1608Metric, F.Cu at (167.2, 96.3)
- added R18: 86k6, Resistor_SMD:R_0603_1608Metric, F.Cu at (167.2, 98.8)
- added R19: 100R, Resistor_SMD:R_0603_1608Metric, F.Cu at (179.5, 129.6)
- added R2: 0R, Resistor_SMD:R_0603_1608Metric, F.Cu at (185.7, 100.7)
- added R20: 1M, Resistor_SMD:R_0603_1608Metric, F.Cu at (179.5, 132.1)
- added R21: 178k, Resistor_SMD:R_0603_1608Metric, F.Cu at (179.5, 134.6)
- added R22: 47k, Resistor_SMD:R_0603_1608Metric, F.Cu at (159.2, 124.6)
- added R23: 10k, Resistor_SMD:R_0603_1608Metric, F.Cu at (159.2, 127.1)
- added R24: 47k, Resistor_SMD:R_0603_1608Metric, F.Cu at (159.2, 129.6)
- added R25: 10k, Resistor_SMD:R_0603_1608Metric, F.Cu at (159.2, 132.1)
- added R26: 47k, Resistor_SMD:R_0603_1608Metric, F.Cu at (159.2, 134.6)
- added R27: 10k, Resistor_SMD:R_0603_1608Metric, F.Cu at (159.2, 137.1)
- added R3: 5k1, Resistor_SMD:R_0603_1608Metric, F.Cu at (63.2, 52.5)
- added R4: 10k, Resistor_SMD:R_0603_1608Metric, F.Cu at (167.2, 50.8)
- added R5: 1k5, Resistor_SMD:R_0603_1608Metric, F.Cu at (63.2, 54.5)
- added R6: 5k1, Resistor_SMD:R_0603_1608Metric, F.Cu at (63.0, 49.5)
- added R7: 130R, Resistor_SMD:R_0603_1608Metric, F.Cu at (167.2, 58.4)
- added R8: 1k, Resistor_SMD:R_0603_1608Metric, F.Cu at (167.2, 60.9)
- added R9: 100R, Resistor_SMD:R_0603_1608Metric, F.Cu at (167.2, 63.4)
- added SW1: SW_SPDT, Button_Switch_SMD:SW_SPDT_PCM12, F.Cu at (184.1, 93.0)
- added SW2: SW_SPDT, Button_Switch_SMD:SW_SPDT_PCM12, F.Cu at (174.2, 84.1)
- added SW3: SW_SPST, Button_Switch_SMD:SW_SPST_B3U-1000P, F.Cu at (164.1, 118.0)
- added SW4: SW_SPST, Button_Switch_SMD:SW_SPST_B3U-1000P, F.Cu at (164.1, 122.3)
- added SW5: SW_SPST, Button_Switch_SMD:SW_SPST_B3U-1000P, F.Cu at (164.1, 126.7)
- added TP1: TestPoint, TestPoint:TestPoint_Pad_D2.5mm, F.Cu at (181.5, 99.2)
- added TP10: TestPoint, TestPoint:TestPoint_Pad_D2.5mm, F.Cu at (185.2, 78.9)
- added TP11: TestPoint, TestPoint:TestPoint_Pad_D2.5mm, F.Cu at (173.6, 109.8)
- added TP2: TestPoint, TestPoint:TestPoint_Pad_D2.5mm, F.Cu at (181.5, 103.8)
- added TP3: TestPoint, TestPoint:TestPoint_Pad_D2.5mm, F.Cu at (171.5, 74.3)
- added TP4: TestPoint, TestPoint:TestPoint_Pad_D2.5mm, F.Cu at (171.5, 78.9)
- added TP5: TestPoint, TestPoint:TestPoint_Pad_D2.5mm, F.Cu at (176.1, 74.3)
- added TP6: TestPoint, TestPoint:TestPoint_Pad_D2.5mm, F.Cu at (176.1, 78.9)
- added TP7: TestPoint, TestPoint:TestPoint_Pad_D2.5mm, F.Cu at (180.6, 74.3)
- added TP8: TestPoint, TestPoint:TestPoint_Pad_D2.5mm, F.Cu at (180.6, 78.9)
- added TP9: TestPoint, TestPoint:TestPoint_Pad_D2.5mm, F.Cu at (185.2, 74.3)
- added U1: STM32F103RCT6, Package_QFP:LQFP-64_10x10mm_P0.5mm, F.Cu at (48.9, 51.5)
- added U2: LD39015M33R, Package_TO_SOT_SMD:SOT-23-5, F.Cu at (186.5, 83.4)
- added U3: TPS63000, Package_SON:Texas_DRC0010J_ThermalVias, F.Cu at (184.0, 121.3)
- added U4: M74HC14YRM13TR, Package_SO:SOIC-14_3.9x8.7mm_P1.27mm, F.Cu at (171.3, 120.9)
- added Y1: 16MHz, Crystal:Crystal_SMD_3225-4Pin_3.2x2.5mm, F.Cu at (31.5, 51.0)
