File: hw/ShotClockProject/LipoBattAndCharger.kicad_sch (KiCad schematic)
At the start: 21 parts, among them IC1 TP4056-42-ESOP8_Rearanged, J2 Conn_01x02_Pin, J8 Conn_01x03_Pin, J9 Conn_01x03_Pin, Q1 Q_PMOS_SGD

Commit message: Finished footprint selection & updated design doc
Chosen all footprints
Updated design doc with part link & part selection reasons
Parts:
- C12, C13: value 10uF -> 10u; footprint Capacitor_SMD:C_0402_1005Metric -> Capacitor_SMD:C_0603_1608Metric
- C12: value 100nF -> 100n; footprint Capacitor_SMD:C_0402_1005Metric -> Capacitor_SMD:C_0603_1608Metric
- J2: footprint (none) -> Connector_PinHeader_2.54mm:PinHeader_1x02_P2.54mm_Vertical_SMD_Pin1Left
- J8: footprint (none) -> Connector_PinHeader_1.00mm:PinHeader_1x03_P1.00mm_Vertical_SMD_Pin1Left
- J9: footprint (none) -> Connector_PinHeader_2.54mm:PinHeader_1x03_P2.54mm_Vertical_SMD_Pin1Left
- NT1: footprint (none) -> NetTie:NetTie-2_SMD_Pad2.0mm
- Q1: footprint (none) -> Package_TO_SOT_SMD:SOT-23
- R19, R20, R3, R4, R5, R6: footprint (none) -> Resistor_SMD:R_0603_1608Metric
- R7: value R? -> 1k; footprint (none) -> Resistor_SMD:R_0603_1608Metric
- TP4: footprint (none) -> TestPoint:TestPoint_Pad_D2.5mm
Changed lines of the file:
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@@
       (effects (font (size 1.27 1.27)))
     )
-    (property "Footprint" "" (at 151.13 110.49 0)
+    (property "Footprint" "Connector_PinHeader_2.54mm:PinHeader_1x03_P2.54mm_Vertical_SMD_Pin1Left" (at 151.13 110.49 0)
       (effects (font (size 1.27 1.27)) hide)
     )
@@
       (effects (font (size 1.27 1.27)))
     )
-    (property "Footprint" "" (at 56.388 57.15 90)
+    (property "Footprint" "Resistor_SMD:R_0603_1608Metric" (at 56.388 57.15 90)
       (effects (font (size 1.27 1.27)) hide)
     )
@@
       (effects (font (size 1.27 1.27)))
     )
-    (property "Footprint" "" (at 34.29 111.76 0)
+    (property "Footprint" "Connector_PinHeader_1.00mm:PinHeader_1x03_P1.00mm_Vertical_SMD_Pin1Left" (at 34.29 111.76 0)
       (effects (font (size 1.27 1.27)) hide)
     )
@@
       (effects (font (size 1.27 1.27)))
     )
-    (property "Footprint" "" (at 107.95 110.49 0)
+    (property "Footprint" "Connector_PinHeader_2.54mm:PinHeader_1x02_P2.54mm_Vertical_SMD_Pin1Left" (at 107.95 110.49 0)
       (effects (font (size 1.27 1.27)) hide)
     )
@@
       (effects (font (size 1.27 1.27)) (justify left))
     )
-    (property "Value" "10uF" (at 146.05 67.31 0)
-      (effects (font (size 1.27 1.27)) (justify left))
-    )
-    (property "Footprint" "Capacitor_SMD:C_0402_1005Metric" (at 143.2052 69.85 0)
+    (property "Value" "10u" (at 146.05 67.31 0)
+      (effects (font (size 1.27 1.27)) (justify left))
+    )
+    (property "Footprint" "Capacitor_SMD:C_0603_1608Metric" (at 143.2052 69.85 0)
       (effects (font (size 1.27 1.27)) hide)
     )
@@
       (effects (font (size 1.27 1.27)))
     )
-    (property "Footprint" "" (at 147.32 74.93 0)
+    (property "Footprint" "NetTie:NetTie-2_SMD_Pad2.0mm" (at 147.32 74.93 0)
       (effects (font (size 1.27 1.27)) hide)
     )
@@
       (effects (font (size 1.27 1.27)))
     )
-    (property "Footprint" "" (at 64.262 119.38 90)
+    (property "Footprint" "Resistor_SMD:R_0603_1608Metric" (at 64.262 119.38 90)
       (effects (font (size 1.27 1.27)) hide)
     )
@@
       (effects (font (size 1.27 1.27)) (justify left))
     )
-    (property "Footprint" "" (at 74.168 40.64 90)
+    (property "Footprint" "Resistor_SMD:R_0603_1608Metric" (at 74.168 40.64 90)
       (effects (font (size 1.27 1.27)) hide)
     )
@@
       (effects (font (size 1.27 1.27)))
     )
-    (property "Footprint" "" (at 125.222 71.12 90)
+    (property "Footprint" "Resistor_SMD:R_0603_1608Metric" (at 125.222 71.12 90)
       (effects (font (size 1.27 1.27)) hide)
     )
@@
       (effects (font (size 1.27 1.27)) (justify left))
     )
-    (property "Footprint" "" (at 236.22 54.61 0)
+    (property "Footprint" "TestPoint:TestPoint_Pad_D2.5mm" (at 236.22 54.61 0)
       (effects (font (size 1.27 1.27)) hide)
     )
@@
       (effects (font (size 1.27 1.27)))
     )
-    (property "Footprint" "" (at 64.262 105.41 90)
+    (property "Footprint" "Resistor_SMD:R_0603_1608Metric" (at 64.262 105.41 90)
       (effects (font (size 1.27 1.27)) hide)
     )
@@
       (effects (font (size 1.27 1.27)))
     )
-    (property "Footprint" "" (at 162.56 63.5 0)
+    (property "Footprint" "Package_TO_SOT_SMD:SOT-23" (at 162.56 63.5 0)
       (effects (font (size 1.27 1.27)) hide)
     )
@@
       (effects (font (size 1.27 1.27)) (justify left))
     )
-    (property "Footprint" "" (at 219.202 48.26 90)
+    (property "Footprint" "Resistor_SMD:R_0603_1608Metric" (at 219.202 48.26 90)
       (effects (font (size 1.27 1.27)) hide)
     )
@@
   (symbol (lib_id "Device:C") (at 44.45 49.53 0) (mirror y) (unit 1)
     (in_bom yes) (on_board yes) (dnp no) (fields_autoplaced)
-    (property "Reference" "C13" (at 40.64 48.26 0)
-      (effects (font (size 1.27 1.27)) (justify left))
-    )
-    (property "Value" "10uF" (at 40.64 50.8 0)
-      (effects (font (size 1.27 1.27)) (justify left))
-    )
-    (property "Footprint" "Capacitor_SMD:C_0402_1005Metric" (at 43.4848 53.34 0)
+    (property "Reference" "C13" (at 48.26 48.26 0)
+      (effects (font (size 1.27 1.27)) (justify right))
+    )
+    (property "Value" "10u" (at 48.26 50.8 0)
+      (effects (font (size 1.27 1.27)) (justify right))
+    )
+    (property "Footprint" "Capacitor_SMD:C_0603_1608Metric" (at 43.4848 53.34 0)
       (effects (font (size 1.27 1.27)) hide)
     )
@@
       (effects (font (size 1.27 1.27)))
     )
-    (property "Footprint" "" (at 65.278 57.15 90)
+    (property "Footprint" "Resistor_SMD:R_0603_1608Metric" (at 65.278 57.15 90)
       (effects (font (size 1.27 1.27)) hide)
     )
@@
       (effects (font (size 1.27 1.27)) (justify right))
     )
-    (property "Value" "R?" (at 162.56 46.99 0)
+    (property "Value" "1k" (at 162.56 46.99 0)
       (effects (font (size 1.27 1.27)) (justify right))
     )
-    (property "Footprint" "" (at 161.798 45.72 90)
+    (property "Footprint" "Resistor_SMD:R_0603_1608Metric" (at 161.798 45.72 90)
       (effects (font (size 1.27 1.27)) hide)
     )
@@
       (effects (font (size 1.27 1.27)) (justify left))
     )
-    (property "Value" "100nF" (at 234.95 62.23 0)
-      (effects (font (size 1.27 1.27)) (justify left))
-    )
-    (property "Footprint" "Capacitor_SMD:C_0402_1005Metric" (at 232.1052 64.77 0)
+    (property "Value" "100n" (at 234.95 62.23 0)
+      (effects (font (size 1.27 1.27)) (justify left))
+    )
+    (property "Footprint" "Capacitor_SMD:C_0603_1608Metric" (at 232.1052 64.77 0)
       (effects (font (size 1.27 1.27)) hide)
     )
@@
       (effects (font (size 1.27 1.27)) (justify left))
     )
-    (property "Footprint" "" (at 219.202 60.96 90)
-      (effects (font (size 1.27 1.27)) hide)
-    )
+    (property "Footprint" "Resistor_SMD:R_0603_1608Metric" (at 219.202 60.96 90)
+      (effects (font (size 1.27 1.27)) hide)
+    )

Commit message: Renamed references
Parts:
- renumbered J8 to J4, J2 to J5, J9 to J6, R19 to R12, R20 to R15
Other:
- note added: "Rprog is 1k2, because that is the max value the datasheet shows (or should I be able to extrapolate the R values to get a higher charge current?) The batteries I want to use (and have at home), are 1500mAh. But charging 1500mAh with 0.66C should also be fine I guess? R1 and R2 calculations are in attached PDF file."
- note removed: "R4 is 1k2, because that is the max value the datasheet shows (or should I be able to extrapolate the R values to get a higher charge current?) The batteries I want to use (and have at home), are 1500mAh. But charging 1500mAh with 0.66C should also be fine I guess? R1 and R2 calculations are in attached PDF file."
- moved on the sheet: J5, J6

Commit message: Changed footprint
To horizontal 2.54 connectors
and started on rough layout
Parts:
- C12: footprint Capacitor_SMD:C_0603_1608Metric -> Capacitor_SMD:C_0402_1005Metric
- J4: footprint Connector_PinHeader_1.00mm:PinHeader_1x03_P1.00mm_Vertical_SMD_Pin1Left -> Connector_PinHeader_1.00mm:PinHeader_1x03_P1.00mm_Horizontal
- J5: footprint Connector_PinHeader_2.54mm:PinHeader_1x02_P2.54mm_Vertical_SMD_Pin1Left -> Connector_PinHeader_2.54mm:PinHeader_1x02_P2.54mm_Horizontal
- J6: footprint Connector_PinHeader_2.54mm:PinHeader_1x03_P2.54mm_Vertical_SMD_Pin1Left -> Connector_PinHeader_2.54mm:PinHeader_1x03_P2.54mm_Horizontal
- R12, R15, R3, R4, R5, R6, R7: footprint Resistor_SMD:R_0603_1608Metric -> Resistor_SMD:R_0402_1005Metric
Changed lines of the file:
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@@
       (effects (font (size 1.27 1.27)))
     )
-    (property "Footprint" "Connector_PinHeader_2.54mm:PinHeader_1x03_P2.54mm_Vertical_SMD_Pin1Left" (at 154.94 118.11 0)
+    (property "Footprint" "Connector_PinHeader_2.54mm:PinHeader_1x03_P2.54mm_Horizontal" (at 154.94 118.11 0)
       (effects (font (size 1.27 1.27)) hide)
     )
@@
       (effects (font (size 1.27 1.27)))
     )
-    (property "Footprint" "Resistor_SMD:R_0603_1608Metric" (at 56.388 57.15 90)
+    (property "Footprint" "Resistor_SMD:R_0402_1005Metric" (at 56.388 57.15 90)
       (effects (font (size 1.27 1.27)) hide)
     )
@@
       (effects (font (size 1.27 1.27)))
     )
-    (property "Footprint" "Connector_PinHeader_1.00mm:PinHeader_1x03_P1.00mm_Vertical_SMD_Pin1Left" (at 34.29 111.76 0)
+    (property "Footprint" "Connector_PinHeader_1.00mm:PinHeader_1x03_P1.00mm_Horizontal" (at 34.29 111.76 0)
       (effects (font (size 1.27 1.27)) hide)
     )
@@
       (effects (font (size 1.27 1.27)))
     )
-    (property "Footprint" "Connector_PinHeader_2.54mm:PinHeader_1x02_P2.54mm_Vertical_SMD_Pin1Left" (at 109.22 113.03 0)
+    (property "Footprint" "Connector_PinHeader_2.54mm:PinHeader_1x02_P2.54mm_Horizontal" (at 109.22 113.03 0)
       (effects (font (size 1.27 1.27)) hide)
     )
@@
       (effects (font (size 1.27 1.27)))
     )
-    (property "Footprint" "Resistor_SMD:R_0603_1608Metric" (at 64.262 119.38 90)
+    (property "Footprint" "Resistor_SMD:R_0402_1005Metric" (at 64.262 119.38 90)
       (effects (font (size 1.27 1.27)) hide)
     )
@@
       (effects (font (size 1.27 1.27)) (justify left))
     )
-    (property "Footprint" "Resistor_SMD:R_0603_1608Metric" (at 74.168 40.64 90)
+    (property "Footprint" "Resistor_SMD:R_0402_1005Metric" (at 74.168 40.64 90)
       (effects (font (size 1.27 1.27)) hide)
     )
@@
       (effects (font (size 1.27 1.27)))
     )
-    (property "Footprint" "Resistor_SMD:R_0603_1608Metric" (at 125.222 71.12 90)
+    (property "Footprint" "Resistor_SMD:R_0402_1005Metric" (at 125.222 71.12 90)
       (effects (font (size 1.27 1.27)) hide)
     )
@@
       (effects (font (size 1.27 1.27)))
     )
-    (property "Footprint" "Resistor_SMD:R_0603_1608Metric" (at 64.262 105.41 90)
+    (property "Footprint" "Resistor_SMD:R_0402_1005Metric" (at 64.262 105.41 90)
       (effects (font (size 1.27 1.27)) hide)
     )
@@
       (effects (font (size 1.27 1.27)) (justify left))
     )
-    (property "Footprint" "Resistor_SMD:R_0603_1608Metric" (at 219.202 48.26 90)
+    (property "Footprint" "Resistor_SMD:R_0402_1005Metric" (at 219.202 48.26 90)
       (effects (font (size 1.27 1.27)) hide)
     )
@@
       (effects (font (size 1.27 1.27)))
     )
-    (property "Footprint" "Resistor_SMD:R_0603_1608Metric" (at 65.278 57.15 90)
+    (property "Footprint" "Resistor_SMD:R_0402_1005Metric" (at 65.278 57.15 90)
       (effects (font (size 1.27 1.27)) hide)
     )
@@
       (effects (font (size 1.27 1.27)) (justify right))
     )
-    (property "Footprint" "Resistor_SMD:R_0603_1608Metric" (at 161.798 45.72 90)
+    (property "Footprint" "Resistor_SMD:R_0402_1005Metric" (at 161.798 45.72 90)
       (effects (font (size 1.27 1.27)) hide)
     )
@@
       (effects (font (size 1.27 1.27)) (justify left))
     )
-    (property "Footprint" "Capacitor_SMD:C_0603_1608Metric" (at 232.1052 64.77 0)
+    (property "Footprint" "Capacitor_SMD:C_0402_1005Metric" (at 232.1052 64.77 0)
       (effects (font (size 1.27 1.27)) hide)
     )
@@
       (effects (font (size 1.27 1.27)) (justify left))
     )
-    (property "Footprint" "Resistor_SMD:R_0603_1608Metric" (at 219.202 60.96 90)
-      (effects (font (size 1.27 1.27)) hide)
-    )
+    (property "Footprint" "Resistor_SMD:R_0402_1005Metric" (at 219.202 60.96 90)
+      (effects (font (size 1.27 1.27)) hide)
+    )
