File: hw/ShotClockProject/LipoBattAndCharger.kicad_sch (KiCad schematic)
At the start: 28 parts, among them IC1 TP4056-42-ESOP8_Rearanged, J4 SM03B-SRSS-TB(LF)(SN)(P), J5 Conn_01x02_Pin, J6 Conn_01x03_Pin, Q1 Q_NPN_BCE, Q1 Q_PMOS_SGD

Commit message: Added LCSC Part number
Renamed output folders
Created first output files for REV1
Parts:
- C12, C13: LCSC Part (none) -> C96446; LCSC Part # (none) -> C96446
- C12: LCSC Part (none) -> C57112; LCSC Part # (none) -> C57112
- C12: LCSC Part (none) -> C1525; LCSC Part # (none) -> C1525
- D1: LCSC Part (none) -> C128250; LCSC Part # (none) -> C128250
- D2: LCSC Part (none) -> C72043; LCSC Part # (none) -> C72043
- IC1: LCSC Part (none) -> C725790; LCSC Part # (none) -> C725790
- J4: LCSC Part # (none) -> C160403
- J5: LCSC Part (none) -> C225269; LCSC Part # (none) -> C225269
- J6: LCSC Part (none) -> C92159; LCSC Part # (none) -> C92159
- Q1: LCSC Part (none) -> C111113; LCSC Part # (none) -> C111113
- Q1: LCSC Part (none) -> C33903; LCSC Part # (none) -> C33903
- R14, R20: LCSC Part (none) -> C144787; LCSC Part # (none) -> C144787
- R2, R5, R6: LCSC Part (none) -> C105637; LCSC Part # (none) -> C105637
- R2: LCSC Part (none) -> C25744; LCSC Part # (none) -> C25744
- R2: LCSC Part (none) -> C25741; LCSC Part # (none) -> C25741
- R3: LCSC Part (none) -> C27147; LCSC Part # (none) -> C27147
- R4: LCSC Part (none) -> C852935; LCSC Part # (none) -> C852935
- R4: LCSC Part (none) -> C25862; LCSC Part # (none) -> C25862
- R4: LCSC Part (none) -> C25900; LCSC Part # (none) -> C25900
Changed lines of the file:
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@@
+      (effects (font (size 1.27 1.27)) hide)
+    )
+    (property "LCSC Part #" "C92159" (at 154.94 118.11 0)
+      (effects (font (size 1.27 1.27)) hide)
+    )
+    (property "LCSC Part" "C92159" (at 154.94 118.11 0)
       (effects (font (size 1.27 1.27)) hide)
     )
@@
       (effects (font (size 1.27 1.27)) hide)
     )
+    (property "LCSC Part #" "C111113" (at 166.37 67.31 0)
+      (effects (font (size 1.27 1.27)) hide)
+    )
+    (property "LCSC Part" "C111113" (at 166.37 67.31 0)
+      (effects (font (size 1.27 1.27)) hide)
+    )
     (pin "1")
     (pin "2")
@@
       (effects (font (size 1.27 1.27)) hide)
     )
+    (property "LCSC Part #" "C105637" (at 41.91 52.07 0)
+      (effects (font (size 1.27 1.27)) hide)
+    )
+    (property "LCSC Part" "C105637" (at 41.91 52.07 0)
+      (effects (font (size 1.27 1.27)) hide)
+    )
     (pin "1")
     (pin "2")
@@
     )
     (property "Datasheet" "~" (at 152.4 54.61 0)
+      (effects (font (size 1.27 1.27)) hide)
+    )
+    (property "LCSC Part #" "C105637" (at 152.4 54.61 0)
+      (effects (font (size 1.27 1.27)) hide)
+    )
+    (property "LCSC Part" "C105637" (at 152.4 54.61 0)
       (effects (font (size 1.27 1.27)) hide)
     )
@@
       (effects (font (size 1.27 1.27)) hide)
     )
+    (property "LCSC Part #" "C25744" (at 177.8 71.12 0)
+      (effects (font (size 1.27 1.27)) hide)
+    )
+    (property "LCSC Part" "C25744" (at 177.8 71.12 0)
+      (effects (font (size 1.27 1.27)) hide)
+    )
     (pin "1")
     (pin "2")
@@
       (effects (font (size 1.27 1.27)) hide)
     )
-    (property "LCSC Part" "C160403" (at 34.29 134.62 0)
-      (effects (font (size 1.27 1.27)) hide)
-    )
     (property "JLC Part" "Extended Part" (at 34.29 137.16 0)
+      (effects (font (size 1.27 1.27)) hide)
+    )
+    (property "LCSC Part #" "C160403" (at 34.29 111.76 0)
+      (effects (font (size 1.27 1.27)) hide)
+    )
+    (property "LCSC Part" "C160403" (at 34.29 111.76 0)
       (effects (font (size 1.27 1.27)) hide)
     )
@@
       (effects (font (size 1.27 1.27)) hide)
     )
+    (property "LCSC Part #" "C33903" (at 186.69 52.07 0)
+      (effects (font (size 1.27 1.27)) hide)
+    )
+    (property "LCSC Part" "C33903" (at 186.69 52.07 0)
+      (effects (font (size 1.27 1.27)) hide)
+    )
     (pin "1")
     (pin "2")
@@
       (effects (font (size 1.27 1.27)) hide)
     )
+    (property "LCSC Part #" "C72043" (at 41.91 43.18 0)
+      (effects (font (size 1.27 1.27)) hide)
+    )
+    (property "LCSC Part" "C72043" (at 41.91 43.18 0)
+      (effects (font (size 1.27 1.27)) hide)
+    )
     (pin "1")
     (pin "2")
@@
       (effects (font (size 1.27 1.27)) hide)
     )
+    (property "LCSC Part #" "C225269" (at 109.22 113.03 0)
+      (effects (font (size 1.27 1.27)) hide)
+    )
+    (property "LCSC Part" "C225269" (at 109.22 113.03 0)
+      (effects (font (size 1.27 1.27)) hide)
+    )
     (pin "1")
     (pin "2")
@@
     )
     (property "Datasheet" "~" (at 121.92 60.96 0)
+      (effects (font (size 1.27 1.27)) hide)
+    )
+    (property "LCSC Part #" "C96446" (at 121.92 60.96 0)
+      (effects (font (size 1.27 1.27)) hide)
+    )
+    (property "LCSC Part" "C96446" (at 121.92 60.96 0)
       (effects (font (size 1.27 1.27)) hide)
     )
@@
       (effects (font (size 1.27 1.27)) hide)
     )
+    (property "LCSC Part #" "" (at 127 69.85 0)
+      (effects (font (size 1.27 1.27)) hide)
+    )
+    (property "LCSC Part" "" (at 127 69.85 0)
+      (effects (font (size 1.27 1.27)) hide)
+    )
     (pin "1")
     (pin "2")
@@
       (effects (font (size 1.27 1.27)) hide)
     )
+    (property "LCSC Part #" "C852935" (at 66.04 119.38 0)
+      (effects (font (size 1.27 1.27)) hide)
+    )
+    (property "LCSC Part" "C852935" (at 66.04 119.38 0)
+      (effects (font (size 1.27 1.27)) hide)
+    )
     (pin "1")
     (pin "2")
@@
       (effects (font (size 1.27 1.27)) hide)
     )
+    (property "LCSC Part #" "C27147" (at 59.69 35.56 0)
+      (effects (font (size 1.27 1.27)) hide)
+    )
+    (property "LCSC Part" "C27147" (at 59.69 35.56 0)
+      (effects (font (size 1.27 1.27)) hide)
+    )
     (pin "1")
     (pin "2")
@@
       (effects (font (size 1.27 1.27)) hide)
     )
+    (property "LCSC Part #" "C57112" (at 143.51 71.12 0)
+      (effects (font (size 1.27 1.27)) hide)
+    )
+    (property "LCSC Part" "C57112" (at 143.51 71.12 0)
+      (effects (font (size 1.27 1.27)) hide)
+    )
     (pin "1")
     (pin "2")
@@
       (effects (font (size 1.27 1.27)) hide)
     )
+    (property "LCSC Part #" "C25862" (at 114.3 66.04 0)
+      (effects (font (size 1.27 1.27)) hide)
+    )
+    (property "LCSC Part" "C25862" (at 114.3 66.04 0)
+      (effects (font (size 1.27 1.27)) hide)
+    )
     (pin "1")
     (pin "2")
@@
     )
     (property "Datasheet" "~" (at 248.92 55.88 0)
+      (effects (font (size 1.27 1.27)) hide)
+    )
+    (property "LCSC Part #" "" (at 243.84 55.88 0)
+      (effects (font (size 1.27 1.27)) hide)
+    )
+    (property "LCSC Part" "" (at 243.84 55.88 0)
       (effects (font (size 1.27 1.27)) hide)
     )
@@
       (effects (font (size 1.27 1.27)) hide)
     )
+    (property "LCSC Part #" "C25741" (at 177.8 54.61 0)
+      (effects (font (size 1.27 1.27)) hide)
+    )
+    (property "LCSC Part" "C25741" (at 177.8 54.61 0)
+      (effects (font (size 1.27 1.27)) hide)
+    )
     (pin "1")
     (pin "2")
@@
       (effects (font (size 1.27 1.27)) hide)
     )
+    (property "LCSC Part #" "C25900" (at 66.04 105.41 0)
+      (effects (font (size 1.27 1.27)) hide)
+    )
+    (property "LCSC Part" "C25900" (at 66.04 105.41 0)
+      (effects (font (size 1.27 1.27)) hide)
+    )
     (pin "1")
     (pin "2")
@@
     )
     (property "Datasheet" "~" (at 50.8 43.18 0)
+      (effects (font (size 1.27 1.27)) hide)
+    )
+    (property "LCSC Part #" "C128250" (at 50.8 43.18 0)
+      (effects (font (size 1.27 1.27)) hide)
+    )
+    (property "LCSC Part" "C128250" (at 50.8 43.18 0)
       (effects (font (size 1.27 1.27)) hide)
     )
@@
     (property "Arrow Price/Stock" "" (at 71.12 1050.8 0)
       (effects (font (size 1.27 1.27)) (justify left top) hide)
+    )
+    (property "LCSC Part #" "C725790" (at 97.79 55.88 0)
+      (effects (font (size 1.27 1.27)) hide)
+    )
+    (property "LCSC Part" "C725790" (at 97.79 55.88 0)
+      (effects (font (size 1.27 1.27)) hide)
     )
     (pin "1")
@@
       (effects (font (size 1.27 1.27)) hide)
     )
+    (property "LCSC Part #" "C144787" (at 233.68 49.53 0)
+      (effects (font (size 1.27 1.27)) hide)
+    )
+    (property "LCSC Part" "C144787" (at 233.68 49.53 0)
+      (effects (font (size 1.27 1.27)) hide)
+    )
     (pin "1")
     (pin "2")
@@
       (effects (font (size 1.27 1.27)) hide)
     )
+    (property "LCSC Part #" "C96446" (at 31.75 44.45 0)
+      (effects (font (size 1.27 1.27)) hide)
+    )
+    (property "LCSC Part" "C96446" (at 31.75 44.45 0)
+      (effects (font (size 1.27 1.27)) hide)
+    )
     (pin "1")
     (pin "2")
@@
     )
     (property "Datasheet" "~" (at 168.91 54.61 0)
+      (effects (font (size 1.27 1.27)) hide)
+    )
+    (property "LCSC Part #" "C105637" (at 168.91 54.61 0)
+      (effects (font (size 1.27 1.27)) hide)
+    )
+    (property "LCSC Part" "C105637" (at 168.91 54.61 0)
       (effects (font (size 1.27 1.27)) hide)
     )
@@
       (effects (font (size 1.27 1.27)) hide)
     )
+    (property "LCSC Part #" "C111113" (at 184.15 67.31 0)
+      (effects (font (size 1.27 1.27)) hide)
+    )
+    (property "LCSC Part" "C111113" (at 184.15 67.31 0)
+      (effects (font (size 1.27 1.27)) hide)
+    )
     (pin "1")
     (pin "2")
@@
       (effects (font (size 1.27 1.27)) hide)
     )
+    (property "LCSC Part #" "C105637" (at 50.8 52.07 0)
+      (effects (font (size 1.27 1.27)) hide)
+    )
+    (property "LCSC Part" "C105637" (at 50.8 52.07 0)
+      (effects (font (size 1.27 1.27)) hide)
+    )
     (pin "1")
     (pin "2")
@@
       (effects (font (size 1.27 1.27)) hide)
     )
+    (property "LCSC Part #" "C1525" (at 243.84 62.23 0)
+      (effects (font (size 1.27 1.27)) hide)
+    )
+    (property "LCSC Part" "C1525" (at 243.84 62.23 0)
+      (effects (font (size 1.27 1.27)) hide)
+    )
     (pin "1")
     (pin "2")
@@
     )
     (property "Datasheet" "~" (at 152.4 71.12 0)
+      (effects (font (size 1.27 1.27)) hide)
+    )
+    (property "LCSC Part #" "C25744" (at 152.4 71.12 0)
+      (effects (font (size 1.27 1.27)) hide)
+    )
+    (property "LCSC Part" "C25744" (at 152.4 71.12 0)
       (effects (font (size 1.27 1.27)) hide)
     )
@@
       (effects (font (size 1.27 1.27)) hide)
     )
+    (property "LCSC Part #" "C144787" (at 233.68 62.23 0)
+      (effects (font (size 1.27 1.27)) hide)
+    )
+    (property "LCSC Part" "C144787" (at 233.68 62.23 0)
+      (effects (font (size 1.27 1.27)) hide)
+    )

Commit message: Start on REV2
Decided to use 16 bit PWM IO expanders for segment displays
Chose another STM, because F1 is out of stock (STM32G070CBT6 now)
Replaced STM32Cube configuration with new config for G0 series.
Updated docs to reflect new parts.
Parts:
- R14, R20: value 1M -> 100k
Changed lines of the file:
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@@
       (effects (font (size 1.27 1.27)) (justify left))
     )
-    (property "Value" "1M" (at 236.22 50.8 0)
+    (property "Value" "100k" (at 236.22 50.8 0)
       (effects (font (size 1.27 1.27)) (justify left))
     )
@@
       (effects (font (size 1.27 1.27)) (justify left))
     )
-    (property "Value" "1M" (at 236.22 63.5 0)
-      (effects (font (size 1.27 1.27)) (justify left))
-    )
+    (property "Value" "100k" (at 236.22 63.5 0)
+      (effects (font (size 1.27 1.27)) (justify left))
+    )

Commit message: Started on integrating new STM32 MCU
Parts:
- renumbered Q1 to Q3, Q1 to Q4
Changed lines of the file:
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@@
   (symbol (lib_id "Device:Q_NPN_BCE") (at 166.37 67.31 0) (unit 1)
     (in_bom yes) (on_board yes) (dnp no)
-    (property "Reference" "Q1" (at 167.64 72.39 0)
+    (property "Reference" "Q3" (at 167.64 72.39 0)
       (effects (font (size 1.27 1.27)) (justify right))
     )
@@
     (instances
       (project "ShotClockProject"
-        (path "/5fd859aa-754d-49c2-9762-3f7ebe3bb64c/d53b1cd8-24cb-4dc0-9a02-0cd96c1f4291"
-          (reference "Q1") (unit 1)
-        )
         (path "/5fd859aa-754d-49c2-9762-3f7ebe3bb64c/d287d155-1951-4d4f-8d6c-570f03bc79f5"
           (reference "Q3") (unit 1)
@@
           (reference "R2") (unit 1)
         )
-        (path "/5fd859aa-754d-49c2-9762-3f7ebe3bb64c/d53b1cd8-24cb-4dc0-9a02-0cd96c1f4291"
-          (reference "R29") (unit 1)
-        )
         (path "/5fd859aa-754d-49c2-9762-3f7ebe3bb64c/d287d155-1951-4d4f-8d6c-570f03bc79f5"
           (reference "R17") (unit 1)
@@
         (path "/5fd859aa-754d-49c2-9762-3f7ebe3bb64c"
           (reference "R2") (unit 1)
-        )
-        (path "/5fd859aa-754d-49c2-9762-3f7ebe3bb64c/d53b1cd8-24cb-4dc0-9a02-0cd96c1f4291"
-          (reference "R29") (unit 1)
         )
         (path "/5fd859aa-754d-49c2-9762-3f7ebe3bb64c/d287d155-1951-4d4f-8d6c-570f03bc79f5"
@@
           (reference "#PWR011") (unit 1)
         )
-        (path "/5fd859aa-754d-49c2-9762-3f7ebe3bb64c/d53b1cd8-24cb-4dc0-9a02-0cd96c1f4291"
-          (reference "#PWR075") (unit 1)
-        )
         (path "/5fd859aa-754d-49c2-9762-3f7ebe3bb64c/d287d155-1951-4d4f-8d6c-570f03bc79f5"
           (reference "#PWR042") (unit 1)
@@
           (reference "TP4") (unit 1)
         )
-        (path "/5fd859aa-754d-49c2-9762-3f7ebe3bb64c/d53b1cd8-24cb-4dc0-9a02-0cd96c1f4291"
-          (reference "TP12") (unit 1)
-        )
         (path "/5fd859aa-754d-49c2-9762-3f7ebe3bb64c/dbe9281d-d28a-4966-832c-4ef9ca7a9777"
           (reference "TP13") (unit 1)
@@
           (reference "R2") (unit 1)
         )
-        (path "/5fd859aa-754d-49c2-9762-3f7ebe3bb64c/d53b1cd8-24cb-4dc0-9a02-0cd96c1f4291"
-          (reference "R29") (unit 1)
-        )
         (path "/5fd859aa-754d-49c2-9762-3f7ebe3bb64c/d287d155-1951-4d4f-8d6c-570f03bc79f5"
           (reference "R19") (unit 1)
@@
         (path "/5fd859aa-754d-49c2-9762-3f7ebe3bb64c"
           (reference "#PWR011") (unit 1)
-        )
-        (path "/5fd859aa-754d-49c2-9762-3f7ebe3bb64c/d53b1cd8-24cb-4dc0-9a02-0cd96c1f4291"
-          (reference "#PWR019") (unit 1)
         )
         (path "/5fd859aa-754d-49c2-9762-3f7ebe3bb64c/d287d155-1951-4d4f-8d6c-570f03bc79f5"
@@
           (reference "IC1") (unit 1)
         )
-        (path "/5fd859aa-754d-49c2-9762-3f7ebe3bb64c/d53b1cd8-24cb-4dc0-9a02-0cd96c1f4291"
-          (reference "IC1") (unit 1)
-        )
       )
     )
@@
           (reference "R2") (unit 1)
         )
-        (path "/5fd859aa-754d-49c2-9762-3f7ebe3bb64c/d53b1cd8-24cb-4dc0-9a02-0cd96c1f4291"
-          (reference "R29") (unit 1)
-        )
         (path "/5fd859aa-754d-49c2-9762-3f7ebe3bb64c/d287d155-1951-4d4f-8d6c-570f03bc79f5"
           (reference "R18") (unit 1)
@@
           (reference "#PWR011") (unit 1)
         )
-        (path "/5fd859aa-754d-49c2-9762-3f7ebe3bb64c/d53b1cd8-24cb-4dc0-9a02-0cd96c1f4291"
-          (reference "#PWR075") (unit 1)
-        )
         (path "/5fd859aa-754d-49c2-9762-3f7ebe3bb64c/d287d155-1951-4d4f-8d6c-570f03bc79f5"
           (reference "#PWR044") (unit 1)
@@
   (symbol (lib_id "Device:Q_NPN_BCE") (at 184.15 67.31 0) (unit 1)
     (in_bom yes) (on_board yes) (dnp no)
-    (property "Reference" "Q1" (at 189.23 66.04 0)
+    (property "Reference" "Q4" (at 189.23 66.04 0)
       (effects (font (size 1.27 1.27)) (justify left))
     )
@@
     (instances
       (project "ShotClockProject"
-        (path "/5fd859aa-754d-49c2-9762-3f7ebe3bb64c/d53b1cd8-24cb-4dc0-9a02-0cd96c1f4291"
-          (reference "Q1") (unit 1)
-        )
         (path "/5fd859aa-754d-49c2-9762-3f7ebe3bb64c/d287d155-1951-4d4f-8d6c-570f03bc79f5"
           (reference "Q4") (unit 1)
@@
   (symbol (lib_id "power:PWR_FLAG") (at 121.92 115.57 180) (unit 1)
     (in_bom yes) (on_board yes) (dnp no) (fields_autoplaced)
-    (property "Reference" "#FLG02" (at 121.92 117.475 0)
+    (property "Reference" "#FLG07" (at 121.92 117.475 0)
       (effects (font (size 1.27 1.27)) hide)
     )
@@
     (instances
       (project "ShotClockProject"
-        (path "/5fd859aa-754d-49c2-9762-3f7ebe3bb64c/d53b1cd8-24cb-4dc0-9a02-0cd96c1f4291"
-          (reference "#FLG02") (unit 1)
-        )
         (path "/5fd859aa-754d-49c2-9762-3f7ebe3bb64c/d287d155-1951-4d4f-8d6c-570f03bc79f5"
           (reference "#FLG07") (unit 1)
@@
           (reference "#PWR011") (unit 1)
         )
-        (path "/5fd859aa-754d-49c2-9762-3f7ebe3bb64c/d53b1cd8-24cb-4dc0-9a02-0cd96c1f4291"
-          (reference "#PWR075") (unit 1)
-        )
         (path "/5fd859aa-754d-49c2-9762-3f7ebe3bb64c/d287d155-1951-4d4f-8d6c-570f03bc79f5"
           (reference "#PWR043") (unit 1)
@@
   (symbol (lib_id "power:PWR_FLAG") (at 121.92 113.03 0) (unit 1)
     (in_bom yes) (on_board yes) (dnp no) (fields_autoplaced)
-    (property "Reference" "#FLG02" (at 121.92 111.125 0)
+    (property "Reference" "#FLG06" (at 121.92 111.125 0)
       (effects (font (size 1.27 1.27)) hide)
     )
@@
     (instances
       (project "ShotClockProject"
-        (path "/5fd859aa-754d-49c2-9762-3f7ebe3bb64c/d53b1cd8-24cb-4dc0-9a02-0cd96c1f4291"
-          (reference "#FLG02") (unit 1)
-        )
         (path "/5fd859aa-754d-49c2-9762-3f7ebe3bb64c/d287d155-1951-4d4f-8d6c-570f03bc79f5"
           (reference "#FLG06") (unit 1)
@@
           (reference "R2") (unit 1)
         )
-        (path "/5fd859aa-754d-49c2-9762-3f7ebe3bb64c/d53b1cd8-24cb-4dc0-9a02-0cd96c1f4291"
-          (reference "R29") (unit 1)
-        )
-        (path "/5fd859aa-754d-49c2-9762-3f7ebe3bb64c/d287d155-1951-4d4f-8d6c-570f03bc79f5"
+        (path "/5fd859aa-754d-49c2-9762-3f7ebe3bb64c/d287d155-1951-4d4f-8d6c-570f03bc79f5"
