File: hw/ShotClockProject/LipoBattAndCharger.kicad_sch (KiCad schematic)
At the start: 27 parts, among them IC1 TP4056-42-ESOP8_Rearanged, J3 SM03B-SRSS-TB(LF)(SN)(P), J4 Conn_01x02_Pin, J7 Conn_01x02_Pin, Q1 Q_PMOS_SGD, Q2 Q_NPN_BCE, Q3 Q_NPN_BCE

Commit message: Updated part NBRS for mainboard
Parts:
- C12, C13: LCSC Part C96446 -> C15525
- J4, J7: LCSC Part C225269 -> C492410
Changed lines of the file:
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@@
-      (effects (font (size 1.27 1.27)) hide)
-    )
-    (property "LCSC Part #" "" (at 166.37 67.31 0)
       (effects (font (size 1.27 1.27)) hide)
     )
@@
       (effects (font (size 1.27 1.27)) hide)
     )
-    (property "LCSC Part #" "" (at 41.91 52.07 0)
-      (effects (font (size 1.27 1.27)) hide)
-    )
     (property "LCSC Part" "C105637" (at 41.91 52.07 0)
       (effects (font (size 1.27 1.27)) hide)
@@
       (effects (font (size 1.27 1.27)) hide)
     )
-    (property "LCSC Part #" "" (at 152.4 54.61 0)
-      (effects (font (size 1.27 1.27)) hide)
-    )
     (property "LCSC Part" "C105637" (at 152.4 54.61 0)
       (effects (font (size 1.27 1.27)) hide)
@@
     )
     (property "Datasheet" "~" (at 177.8 71.12 0)
-      (effects (font (size 1.27 1.27)) hide)
-    )
-    (property "LCSC Part #" "" (at 177.8 71.12 0)
       (effects (font (size 1.27 1.27)) hide)
     )
@@
     )
     (property "JLC Part" "Extended Part" (at 34.29 137.16 0)
-      (effects (font (size 1.27 1.27)) hide)
-    )
-    (property "LCSC Part #" "" (at 34.29 111.76 0)
       (effects (font (size 1.27 1.27)) hide)
     )
@@
       (effects (font (size 1.27 1.27)) hide)
     )
-    (property "LCSC Part #" "" (at 186.69 52.07 0)
-      (effects (font (size 1.27 1.27)) hide)
-    )
     (property "LCSC Part" "C33903" (at 186.69 52.07 0)
       (effects (font (size 1.27 1.27)) hide)
@@
       (effects (font (size 1.27 1.27)) hide)
     )
-    (property "LCSC Part #" "" (at 41.91 43.18 0)
-      (effects (font (size 1.27 1.27)) hide)
-    )
     (property "LCSC Part" "C72043" (at 41.91 43.18 0)
       (effects (font (size 1.27 1.27)) hide)
@@
       (effects (font (size 1.27 1.27)) hide)
     )
-    (property "LCSC Part #" "" (at 109.22 113.03 0)
-      (effects (font (size 1.27 1.27)) hide)
-    )
-    (property "LCSC Part" "C225269" (at 109.22 113.03 0)
+    (property "LCSC Part" "C492410" (at 109.22 113.03 0)
       (effects (font (size 1.27 1.27)) hide)
     )
@@
       (effects (font (size 1.27 1.27)) hide)
     )
-    (property "LCSC Part #" "" (at 121.92 60.96 0)
-      (effects (font (size 1.27 1.27)) hide)
-    )
-    (property "LCSC Part" "C96446" (at 121.92 60.96 0)
+    (property "LCSC Part" "C15525" (at 121.92 60.96 0)
       (effects (font (size 1.27 1.27)) hide)
     )
@@
       (effects (font (size 1.27 1.27)) hide)
     )
-    (property "LCSC Part #" "" (at 154.94 118.11 0)
-      (effects (font (size 1.27 1.27)) hide)
-    )
-    (property "LCSC Part" "C225269" (at 154.94 118.11 0)
+    (property "LCSC Part" "C492410" (at 154.94 118.11 0)
       (effects (font (size 1.27 1.27)) hide)
     )
@@
       (effects (font (size 1.27 1.27)) hide)
     )
-    (property "LCSC Part #" "" (at 66.04 119.38 0)
-      (effects (font (size 1.27 1.27)) hide)
-    )
     (property "LCSC Part" "C852935" (at 66.04 119.38 0)
       (effects (font (size 1.27 1.27)) hide)
@@
       (effects (font (size 1.27 1.27)) hide)
     )
-    (property "LCSC Part #" "" (at 59.69 35.56 0)
-      (effects (font (size 1.27 1.27)) hide)
-    )
     (property "LCSC Part" "C27147" (at 59.69 35.56 0)
       (effects (font (size 1.27 1.27)) hide)
@@
       (effects (font (size 1.27 1.27)) hide)
     )
-    (property "LCSC Part #" "" (at 143.51 71.12 0)
-      (effects (font (size 1.27 1.27)) hide)
-    )
     (property "LCSC Part" "C15195" (at 143.51 71.12 0)
       (effects (font (size 1.27 1.27)) hide)
@@
       (effects (font (size 1.27 1.27)) hide)
     )
-    (property "LCSC Part #" "" (at 114.3 66.04 0)
-      (effects (font (size 1.27 1.27)) hide)
-    )
     (property "LCSC Part" "C25862" (at 114.3 66.04 0)
       (effects (font (size 1.27 1.27)) hide)
@@
       (effects (font (size 1.27 1.27)) hide)
     )
-    (property "LCSC Part #" "" (at 177.8 54.61 0)
-      (effects (font (size 1.27 1.27)) hide)
-    )
     (property "LCSC Part" "C25741" (at 177.8 54.61 0)
       (effects (font (size 1.27 1.27)) hide)
@@
       (effects (font (size 1.27 1.27)) hide)
     )
-    (property "LCSC Part #" "" (at 66.04 105.41 0)
-      (effects (font (size 1.27 1.27)) hide)
-    )
     (property "LCSC Part" "C25900" (at 66.04 105.41 0)
       (effects (font (size 1.27 1.27)) hide)
@@
     )
     (property "Datasheet" "~" (at 50.8 43.18 0)
-      (effects (font (size 1.27 1.27)) hide)
-    )
-    (property "LCSC Part #" "" (at 50.8 43.18 0)
       (effects (font (size 1.27 1.27)) hide)
     )
@@
     (property "Arrow Price/Stock" "" (at 71.12 1050.8 0)
       (effects (font (size 1.27 1.27)) (justify left top) hide)
-    )
-    (property "LCSC Part #" "" (at 97.79 55.88 0)
-      (effects (font (size 1.27 1.27)) hide)
     )
     (property "LCSC Part" "C725790" (at 97.79 55.88 0)
@@
       (effects (font (size 1.27 1.27)) hide)
     )
-    (property "LCSC Part #" "" (at 233.68 49.53 0)
-      (effects (font (size 1.27 1.27)) hide)
-    )
     (property "LCSC Part" "C25741" (at 233.68 49.53 0)
       (effects (font (size 1.27 1.27)) hide)
@@
       (effects (font (size 1.27 1.27)) hide)
     )
-    (property "LCSC Part #" "" (at 31.75 44.45 0)
-      (effects (font (size 1.27 1.27)) hide)
-    )
-    (property "LCSC Part" "C96446" (at 31.75 44.45 0)
+    (property "LCSC Part" "C15525" (at 31.75 44.45 0)
       (effects (font (size 1.27 1.27)) hide)
     )
@@
       (effects (font (size 1.27 1.27)) hide)
     )
-    (property "LCSC Part #" "" (at 168.91 54.61 0)
-      (effects (font (size 1.27 1.27)) hide)
-    )
     (property "LCSC Part" "C105637" (at 168.91 54.61 0)
       (effects (font (size 1.27 1.27)) hide)
@@
       (effects (font (size 1.27 1.27)) hide)
     )
-    (property "LCSC Part #" "" (at 184.15 67.31 0)
-      (effects (font (size 1.27 1.27)) hide)
-    )
     (property "LCSC Part" "C111113" (at 184.15 67.31 0)
       (effects (font (size 1.27 1.27)) hide)
@@
     )
     (property "Datasheet" "~" (at 50.8 52.07 0)
-      (effects (font (size 1.27 1.27)) hide)
-    )
-    (property "LCSC Part #" "" (at 50.8 52.07 0)
       (effects (font (size 1.27 1.27)) hide)
     )
@@
       (effects (font (size 1.27 1.27)) hide)
     )
-    (property "LCSC Part #" "" (at 243.84 62.23 0)
-      (effects (font (size 1.27 1.27)) hide)
-    )
     (property "LCSC Part" "C1525" (at 243.84 62.23 0)
       (effects (font (size 1.27 1.27)) hide)
@@
       (effects (font (size 1.27 1.27)) hide)
     )
-    (property "LCSC Part #" "" (at 152.4 71.12 0)
-      (effects (font (size 1.27 1.27)) hide)
-    )
     (property "LCSC Part" "C25744" (at 152.4 71.12 0)
       (effects (font (size 1.27 1.27)) hide)
@@
       (effects (font (size 1.27 1.27)) hide)
     )
-    (property "LCSC Part #" "" (at 233.68 62.23 0)
-      (effects (font (size 1.27 1.27)) hide)
-    )
