File: hw/ShotClockProject/SchmittTriggerWithButtons.kicad_sch (KiCad schematic)
At the start: 13 parts, among them SW2 SW_SPST, SW3 SW_SPST, SW4 SW_SPST, U3 M74HC14YRM13TR

Commit message: Fixed all ERC issues
Mainly by placing PWR_FLAGs and NetTies to show KiCAD where the GNDs are connected to each other physically, without them being the same net.
Connections:
- net +3V3 renamed +3.3V
- no-connect marks 0 -> 6
Changed lines of the file:
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@@
     (date "2023-06-28")
     (rev "1")
+    (comment 1 "Author: M. de Waard")
   )
   (junction (at 138.43 77.47) (diameter 0) (color 0 0 0 0)
@@
   (junction (at 138.43 123.19) (diameter 0) (color 0 0 0 0)
   )
+  (no_connect (at 158.75 85.09))
+  (no_connect (at 194.31 90.17))
+  (no_connect (at 194.31 85.09))
+  (no_connect (at 158.75 87.63))
+  (no_connect (at 194.31 87.63))
+  (no_connect (at 158.75 90.17))
   (wire (pts (xy 149.86 82.55) (xy 149.86 123.19))
     (stroke (width 0) (type default))
@@
     (stroke (width 0) (type default))
   )
+  (wire (pts (xy 194.31 72.39) (xy 204.47 72.39))
+    (stroke (width 0) (type default))
+  )
   (wire (pts (xy 138.43 100.33) (xy 147.32 100.33))
     (stroke (width 0) (type default))
@@
     (stroke (width 0) (type default))
   )
-  (wire (pts (xy 196.85 72.39) (xy 194.31 72.39))
-    (stroke (width 0) (type default))
-  )
   (wire (pts (xy 194.31 95.25) (xy 195.58 95.25))
     (stroke (width 0) (type default))
@@
     (stroke (width 0) (type default))
   )
-  (wire (pts (xy 196.85 68.58) (xy 196.85 72.39))
-    (stroke (width 0) (type default))
-  )
   (wire (pts (xy 138.43 123.19) (xy 138.43 127))
     (stroke (width 0) (type default))
@@
   )
   (wire (pts (xy 194.31 80.01) (xy 205.74 80.01))
+    (stroke (width 0) (type default))
+  )
+  (wire (pts (xy 204.47 64.77) (xy 204.47 72.39))
     (stroke (width 0) (type default))
   )
@@
     )
   )
-  (symbol (lib_id "power:+3V3") (at 96.52 64.77 0) (unit 1)
-    (in_bom yes) (on_board yes) (dnp no) (fields_autoplaced)
-    (property "Reference" "#PWR034" (at 96.52 68.58 0)
-      (effects (font (size 1.27 1.27)) hide)
-    )
-    (property "Value" "+3V3" (at 96.52 59.69 0)
+  (symbol (lib_id "Device:R") (at 127 100.33 90) (unit 1)
+    (in_bom yes) (on_board yes) (dnp no)
+    (property "Reference" "R16" (at 127 95.25 90)
+      (effects (font (size 1.27 1.27)))
+    )
+    (property "Value" "10k" (at 127 97.79 90)
+      (effects (font (size 1.27 1.27)))
+    )
+    (property "Footprint" "" (at 127 102.108 90)
+      (effects (font (size 1.27 1.27)) hide)
+    )
+    (property "Datasheet" "~" (at 127 100.33 0)
+      (effects (font (size 1.27 1.27)) hide)
+    )
+    (pin "1")
+    (pin "2")
+    (instances
+      (project "ShotClockProject"
+        (path "/5fd859aa-754d-49c2-9762-3f7ebe3bb64c/1ce26b90-d7f5-4886-998a-a021d351eec6"
+          (reference "R16") (unit 1)
+        )
+      )
+    )
+  )
+  (symbol (lib_id "Switch:SW_SPST") (at 113.03 129.54 270) (unit 1)
+    (in_bom yes) (on_board yes) (dnp no)
+    (property "Reference" "SW4" (at 115.57 128.27 90)
+      (effects (font (size 1.27 1.27)) (justify left))
+    )
+    (property "Value" "SW_SPST" (at 115.57 130.81 90)
+      (effects (font (size 1.27 1.27)) (justify left))
+    )
+    (property "Footprint" "" (at 113.03 129.54 0)
+      (effects (font (size 1.27 1.27)) hide)
+    )
+    (property "Datasheet" "~" (at 113.03 129.54 0)
+      (effects (font (size 1.27 1.27)) hide)
+    )
+    (pin "1")
+    (pin "2")
+    (instances
+      (project "ShotClockProject"
+        (path "/5fd859aa-754d-49c2-9762-3f7ebe3bb64c/1ce26b90-d7f5-4886-998a-a021d351eec6"
+          (reference "SW4") (unit 1)
+        )
+      )
+    )
+  )
+  (symbol (lib_id "power:+3.3V") (at 96.52 64.77 0) (unit 1)
+    (in_bom yes) (on_board yes) (dnp no)
+    (property "Reference" "#PWR02" (at 96.52 68.58 0)
+      (effects (font (size 1.27 1.27)) hide)
+    )
+    (property "Value" "+3.3V" (at 96.52 60.96 0)
       (effects (font (size 1.27 1.27)))
     )
@@
     (instances
       (project "ShotClockProject"
+        (path "/5fd859aa-754d-49c2-9762-3f7ebe3bb64c"
+          (reference "#PWR02") (unit 1)
+        )
+        (path "/5fd859aa-754d-49c2-9762-3f7ebe3bb64c/d53b1cd8-24cb-4dc0-9a02-0cd96c1f4291"
+          (reference "#PWR06") (unit 1)
+        )
         (path "/5fd859aa-754d-49c2-9762-3f7ebe3bb64c/1ce26b90-d7f5-4886-998a-a021d351eec6"
           (reference "#PWR034") (unit 1)
-        )
-      )
-    )
-  )
-  (symbol (lib_id "Device:R") (at 127 100.33 90) (unit 1)
-    (in_bom yes) (on_board yes) (dnp no)
-    (property "Reference" "R16" (at 127 95.25 90)
-      (effects (font (size 1.27 1.27)))
-    )
-    (property "Value" "10k" (at 127 97.79 90)
-      (effects (font (size 1.27 1.27)))
-    )
-    (property "Footprint" "" (at 127 102.108 90)
-      (effects (font (size 1.27 1.27)) hide)
-    )
-    (property "Datasheet" "~" (at 127 100.33 0)
-      (effects (font (size 1.27 1.27)) hide)
-    )
-    (pin "1")
-    (pin "2")
-    (instances
-      (project "ShotClockProject"
-        (path "/5fd859aa-754d-49c2-9762-3f7ebe3bb64c/1ce26b90-d7f5-4886-998a-a021d351eec6"
-          (reference "R16") (unit 1)
-        )
-      )
-    )
-  )
-  (symbol (lib_id "Switch:SW_SPST") (at 113.03 129.54 270) (unit 1)
-    (in_bom yes) (on_board yes) (dnp no)
-    (property "Reference" "SW4" (at 115.57 128.27 90)
-      (effects (font (size 1.27 1.27)) (justify left))
-    )
-    (property "Value" "SW_SPST" (at 115.57 130.81 90)
-      (effects (font (size 1.27 1.27)) (justify left))
-    )
-    (property "Footprint" "" (at 113.03 129.54 0)
-      (effects (font (size 1.27 1.27)) hide)
-    )
-    (property "Datasheet" "~" (at 113.03 129.54 0)
-      (effects (font (size 1.27 1.27)) hide)
-    )
-    (pin "1")
-    (pin "2")
-    (instances
-      (project "ShotClockProject"
-        (path "/5fd859aa-754d-49c2-9762-3f7ebe3bb64c/1ce26b90-d7f5-4886-998a-a021d351eec6"
-          (reference "SW4") (unit 1)
         )
       )
@@
     )
   )
+  (symbol (lib_id "power:+3.3V") (at 204.47 64.77 0) (unit 1)
+    (in_bom yes) (on_board yes) (dnp no)
+    (property "Reference" "#PWR02" (at 204.47 68.58 0)
+      (effects (font (size 1.27 1.27)) hide)
+    )
+    (property "Value" "+3.3V" (at 204.47 60.96 0)
+      (effects (font (size 1.27 1.27)))
+    )
+    (property "Footprint" "" (at 204.47 64.77 0)
+      (effects (font (size 1.27 1.27)) hide)
+    )
+    (property "Datasheet" "" (at 204.47 64.77 0)
+      (effects (font (size 1.27 1.27)) hide)
+    )
+    (pin "1")
+    (instances
+      (project "ShotClockProject"
+        (path "/5fd859aa-754d-49c2-9762-3f7ebe3bb64c"
+          (reference "#PWR02") (unit 1)
+        )
+        (path "/5fd859aa-754d-49c2-9762-3f7ebe3bb64c/d53b1cd8-24cb-4dc0-9a02-0cd96c1f4291"
+          (reference "#PWR06") (unit 1)
+        )
+        (path "/5fd859aa-754d-49c2-9762-3f7ebe3bb64c/1ce26b90-d7f5-4886-998a-a021d351eec6"
+          (reference "#PWR036") (unit 1)
+        )
+      )
+    )
+  )
   (symbol (lib_id "Device:R") (at 127 77.47 90) (unit 1)
     (in_bom yes) (on_board yes) (dnp no)
@@
         )
       )
-    )
-  )
-  (symbol (lib_id "power:+3V3") (at 196.85 68.58 0) (unit 1)
-    (in_bom yes) (on_board yes) (dnp no) (fields_autoplaced)
-    (property "Reference" "#PWR036" (at 196.85 72.39 0)
-      (effects (font (size 1.27 1.27)) hide)
-    )
-    (property "Value" "+3V3" (at 196.85 63.5 0)
-      (effects (font (size 1.27 1.27)))
-    )
-    (property "Footprint" "" (at 196.85 68.58 0)
-      (effects (font (size 1.27 1.27)) hide)
-    )
-    (property "Datasheet" "" (at 196.85 68.58 0)
-      (effects (font (size 1.27 1.27)) hide)
-    )
-    (pin "1")
-    (instances
-      (project "ShotClockProject"
-        (path "/5fd859aa-754d-49c2-9762-3f7ebe3bb64c/1ce26b90-d7f5-4886-998a-a021d351eec6"
-          (reference "#PWR036") (unit 1)
-        )
-      )

Commit message: Init of SW, changes on HW
SW init STMIDE project
HW Added first few footprints for passive components.
Removed old name .IOC file
Parts:
- C4: footprint (none) -> Capacitor_SMD:C_0402_1005Metric
- U3: footprint SOIC127P600X175-14N -> (none)
Changed lines of the file:
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@@
       (effects (font (size 1.27 1.27)))
     )
-    (property "Footprint" "SOIC127P600X175-14N" (at 176.53 85.09 0)
+    (property "Footprint" "" (at 176.53 85.09 0)
       (effects (font (size 1.27 1.27)) (justify bottom) hide)
     )
@@
       (effects (font (size 1.27 1.27)) (justify left))
     )
-    (property "Footprint" "" (at 139.3952 88.9 0)
+    (property "Footprint" "Capacitor_SMD:C_0402_1005Metric" (at 139.3952 88.9 0)
       (effects (font (size 1.27 1.27)) hide)
     )
@@
       (effects (font (size 1.27 1.27)) (justify left))
     )
-    (property "Footprint" "" (at 139.3952 134.62 0)
+    (property "Footprint" "Capacitor_SMD:C_0402_1005Metric" (at 139.3952 134.62 0)
       (effects (font (size 1.27 1.27)) hide)
     )
@@
       (effects (font (size 1.27 1.27)) (justify left))
     )
-    (property "Footprint" "" (at 139.3952 111.76 0)
-      (effects (font (size 1.27 1.27)) hide)
-    )
+    (property "Footprint" "Capacitor_SMD:C_0402_1005Metric" (at 139.3952 111.76 0)
+      (effects (font (size 1.27 1.27)) hide)
+    )

Commit message: Finished footprint selection & updated design doc
Chosen all footprints
Updated design doc with part link & part selection reasons
Parts:
- C4: footprint Capacitor_SMD:C_0402_1005Metric -> Capacitor_SMD:C_0603_1608Metric
- R13, R14, R15, R16, R17, R18: footprint (none) -> Resistor_SMD:R_0603_1608Metric
- SW2, SW3, SW4: footprint (none) -> Button_Switch_SMD:SW_SPST_B3U-1000P
- U3: footprint (none) -> Package_SO:SOIC-14_3.9x8.7mm_P1.27mm
Changed lines of the file:
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@@
       (effects (font (size 1.27 1.27)) (justify left))
     )
-    (property "Footprint" "" (at 113.03 106.68 0)
+    (property "Footprint" "Button_Switch_SMD:SW_SPST_B3U-1000P" (at 113.03 106.68 0)
       (effects (font (size 1.27 1.27)) hide)
     )
@@
       (effects (font (size 1.27 1.27)))
     )
-    (property "Footprint" "" (at 176.53 85.09 0)
+    (property "Footprint" "Package_SO:SOIC-14_3.9x8.7mm_P1.27mm" (at 176.53 85.09 0)
       (effects (font (size 1.27 1.27)) (justify bottom) hide)
     )
@@
       (effects (font (size 1.27 1.27)) (justify left))
     )
-    (property "Footprint" "Capacitor_SMD:C_0402_1005Metric" (at 139.3952 88.9 0)
+    (property "Footprint" "Capacitor_SMD:C_0603_1608Metric" (at 139.3952 88.9 0)
       (effects (font (size 1.27 1.27)) hide)
     )
@@
       (effects (font (size 1.27 1.27)))
     )
-    (property "Footprint" "" (at 127 102.108 90)
+    (property "Footprint" "Resistor_SMD:R_0603_1608Metric" (at 127 102.108 90)
       (effects (font (size 1.27 1.27)) hide)
     )
@@
       (effects (font (size 1.27 1.27)) (justify left))
     )
-    (property "Footprint" "" (at 113.03 129.54 0)
+    (property "Footprint" "Button_Switch_SMD:SW_SPST_B3U-1000P" (at 113.03 129.54 0)
       (effects (font (size 1.27 1.27)) hide)
     )
@@
       (effects (font (size 1.27 1.27)))
     )
-    (property "Footprint" "" (at 102.87 124.968 90)
+    (property "Footprint" "Resistor_SMD:R_0603_1608Metric" (at 102.87 124.968 90)
       (effects (font (size 1.27 1.27)) hide)
     )
@@
       (effects (font (size 1.27 1.27)))
     )
-    (property "Footprint" "" (at 102.87 79.248 90)
+    (property "Footprint" "Resistor_SMD:R_0603_1608Metric" (at 102.87 79.248 90)
       (effects (font (size 1.27 1.27)) hide)
     )
@@
       (effects (font (size 1.27 1.27)) (justify left))
     )
-    (property "Footprint" "Capacitor_SMD:C_0402_1005Metric" (at 139.3952 134.62 0)
+    (property "Footprint" "Capacitor_SMD:C_0603_1608Metric" (at 139.3952 134.62 0)
       (effects (font (size 1.27 1.27)) hide)
     )
@@
       (effects (font (size 1.27 1.27)))
     )
-    (property "Footprint" "" (at 127 79.248 90)
+    (property "Footprint" "Resistor_SMD:R_0603_1608Metric" (at 127 79.248 90)
       (effects (font (size 1.27 1.27)) hide)
     )
@@
       (effects (font (size 1.27 1.27)))
     )
-    (property "Footprint" "" (at 102.87 102.108 90)
+    (property "Footprint" "Resistor_SMD:R_0603_1608Metric" (at 102.87 102.108 90)
       (effects (font (size 1.27 1.27)) hide)
     )
@@
       (effects (font (size 1.27 1.27)) (justify left))
     )
-    (property "Footprint" "Capacitor_SMD:C_0402_1005Metric" (at 139.3952 111.76 0)
+    (property "Footprint" "Capacitor_SMD:C_0603_1608Metric" (at 139.3952 111.76 0)
       (effects (font (size 1.27 1.27)) hide)
     )
@@
       (effects (font (size 1.27 1.27)))
     )
-    (property "Footprint" "" (at 127 124.968 90)
+    (property "Footprint" "Resistor_SMD:R_0603_1608Metric" (at 127 124.968 90)
       (effects (font (size 1.27 1.27)) hide)
     )
@@
       (effects (font (size 1.27 1.27)) (justify left))
     )
-    (property "Footprint" "" (at 113.03 83.82 0)
-      (effects (font (size 1.27 1.27)) hide)
-    )
+    (property "Footprint" "Button_Switch_SMD:SW_SPST_B3U-1000P" (at 113.03 83.82 0)
+      (effects (font (size 1.27 1.27)) hide)
+    )

Commit message: Renamed references
Parts:
- renumbered R13 to R22, R14 to R23, R15 to R24, R16 to R25, R17 to R26, R18 to R27, SW2 to SW3, SW3 to SW4, SW4 to SW5
Changed lines of the file:
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@@
   (symbol (lib_id "Switch:SW_SPST") (at 113.03 106.68 270) (unit 1)
     (in_bom yes) (on_board yes) (dnp no)
-    (property "Reference" "SW3" (at 115.57 105.41 90)
+    (property "Reference" "SW4" (at 115.57 105.41 90)
       (effects (font (size 1.27 1.27)) (justify left))
     )
@@
       (project "ShotClockProject"
         (path "/5fd859aa-754d-49c2-9762-3f7ebe3bb64c/1ce26b90-d7f5-4886-998a-a021d351eec6"
-          (reference "SW3") (unit 1)
+          (reference "SW4") (unit 1)
         )
       )
@@
         )
         (path "/5fd859aa-754d-49c2-9762-3f7ebe3bb64c/1ce26b90-d7f5-4886-998a-a021d351eec6"
-          (reference "U3") (unit 1)
+          (reference "U4") (unit 1)
         )
       )
@@
         )
         (path "/5fd859aa-754d-49c2-9762-3f7ebe3bb64c/1ce26b90-d7f5-4886-998a-a021d351eec6"
-          (reference "C19") (unit 1)
+          (reference "C22") (unit 1)
         )
       )
@@
   (symbol (lib_id "Device:R") (at 127 100.33 90) (unit 1)
     (in_bom yes) (on_board yes) (dnp no)
-    (property "Reference" "R16" (at 127 95.25 90)
+    (property "Reference" "R25" (at 127 95.25 90)
       (effects (font (size 1.27 1.27)))
     )
@@
       (project "ShotClockProject"
         (path "/5fd859aa-754d-49c2-9762-3f7ebe3bb64c/1ce26b90-d7f5-4886-998a-a021d351eec6"
-          (reference "R16") (unit 1)
+          (reference "R25") (unit 1)
         )
       )
@@
   (symbol (lib_id "Switch:SW_SPST") (at 113.03 129.54 270) (unit 1)
     (in_bom yes) (on_board yes) (dnp no)
-    (property "Reference" "SW4" (at 115.57 128.27 90)
+    (property "Reference" "SW5" (at 115.57 128.27 90)
       (effects (font (size 1.27 1.27)) (justify left))
     )
@@
       (project "ShotClockProject"
         (path "/5fd859aa-754d-49c2-9762-3f7ebe3bb64c/1ce26b90-d7f5-4886-998a-a021d351eec6"
-          (reference "SW4") (unit 1)
+          (reference "SW5") (unit 1)
         )
       )
@@
         )
         (path "/5fd859aa-754d-49c2-9762-3f7ebe3bb64c/1ce26b90-d7f5-4886-998a-a021d351eec6"
-          (reference "#PWR034") (unit 1)
+          (reference "#PWR052") (unit 1)
         )
       )
@@
   (symbol (lib_id "Device:R") (at 102.87 123.19 90) (unit 1)
     (in_bom yes) (on_board yes) (dnp no)
-    (property "Reference" "R17" (at 102.87 118.11 90)
+    (property "Reference" "R26" (at 102.87 118.11 90)
       (effects (font (size 1.27 1.27)))
     )
@@
       (project "ShotClockProject"
         (path "/5fd859aa-754d-49c2-9762-3f7ebe3bb64c/1ce26b90-d7f5-4886-998a-a021d351eec6"
-          (reference "R17") (unit 1)
+          (reference "R26") (unit 1)
         )
       )
@@
   (symbol (lib_id "Device:R") (at 102.87 77.47 90) (unit 1)
     (in_bom yes) (on_board yes) (dnp no)
-    (property "Reference" "R13" (at 102.87 72.39 90)
+    (property "Reference" "R22" (at 102.87 72.39 90)
       (effects (font (size 1.27 1.27)))
     )
@@
       (project "ShotClockProject"
         (path "/5fd859aa-754d-49c2-9762-3f7ebe3bb64c/1ce26b90-d7f5-4886-998a-a021d351eec6"
-          (reference "R13") (unit 1)
+          (reference "R22") (unit 1)
         )
       )
@@
         )
         (path "/5fd859aa-754d-49c2-9762-3f7ebe3bb64c/1ce26b90-d7f5-4886-998a-a021d351eec6"
-          (reference "#PWR037") (unit 1)
+          (reference "#PWR056") (unit 1)
         )
       )
@@
         )
         (path "/5fd859aa-754d-49c2-9762-3f7ebe3bb64c/1ce26b90-d7f5-4886-998a-a021d351eec6"
-          (reference "#PWR039") (unit 1)
+          (reference "#PWR057") (unit 1)
         )
       )
@@
         )
         (path "/5fd859aa-754d-49c2-9762-3f7ebe3bb64c/1ce26b90-d7f5-4886-998a-a021d351eec6"
-          (reference "C21") (unit 1)
+          (reference "C24") (unit 1)
         )
       )
@@
         )
         (path "/5fd859aa-754d-49c2-9762-3f7ebe3bb64c/1ce26b90-d7f5-4886-998a-a021d351eec6"
-          (reference "#PWR041") (unit 1)
+          (reference "#PWR059") (unit 1)
         )
       )
@@
         )
         (path "/5fd859aa-754d-49c2-9762-3f7ebe3bb64c/1ce26b90-d7f5-4886-998a-a021d351eec6"
-          (reference "#PWR036") (unit 1)
+          (reference "#PWR053") (unit 1)
         )
       )
@@
   (symbol (lib_id "Device:R") (at 127 77.47 90) (unit 1)
     (in_bom yes) (on_board yes) (dnp no)
-    (property "Reference" "R14" (at 127 72.39 90)
+    (property "Reference" "R23" (at 127 72.39 90)
       (effects (font (size 1.27 1.27)))
     )
@@
       (project "ShotClockProject"
         (path "/5fd859aa-754d-49c2-9762-3f7ebe3bb64c/1ce26b90-d7f5-4886-998a-a021d351eec6"
-          (reference "R14") (unit 1)
+          (reference "R23") (unit 1)
         )
       )
@@
   (symbol (lib_id "Device:R") (at 102.87 100.33 90) (unit 1)
     (in_bom yes) (on_board yes) (dnp no)
-    (property "Reference" "R15" (at 102.87 95.25 90)
+    (property "Reference" "R24" (at 102.87 95.25 90)
       (effects (font (size 1.27 1.27)))
     )
@@
       (project "ShotClockProject"
         (path "/5fd859aa-754d-49c2-9762-3f7ebe3bb64c/1ce26b90-d7f5-4886-998a-a021d351eec6"
-          (reference "R15") (unit 1)
+          (reference "R24") (unit 1)
         )
       )
@@
         )
         (path "/5fd859aa-754d-49c2-9762-3f7ebe3bb64c/1ce26b90-d7f5-4886-998a-a021d351eec6"
-          (reference "#PWR035") (unit 1)
+          (reference "#PWR054") (unit 1)
         )
       )
@@
         )
         (path "/5fd859aa-754d-49c2-9762-3f7ebe3bb64c/1ce26b90-d7f5-4886-998a-a021d351eec6"
-          (reference "#PWR045") (unit 1)
+          (reference "#PWR060") (unit 1)
         )
       )
@@
         )
         (path "/5fd859aa-754d-49c2-9762-3f7ebe3bb64c/1ce26b90-d7f5-4886-998a-a021d351eec6"
-          (reference "C20") (unit 1)
+          (reference "C23") (unit 1)
         )
       )
@@
         )
         (path "/5fd859aa-754d-49c2-9762-3f7ebe3bb64c/1ce26b90-d7f5-4886-998a-a021d351eec6"
-          (reference "#PWR043") (unit 1)
+          (reference "#PWR055") (unit 1)
         )
       )
@@
         )
         (path "/5fd859aa-754d-49c2-9762-3f7ebe3bb64c/1ce26b90-d7f5-4886-998a-a021d351eec6"
-          (reference "#PWR044") (unit 1)
+          (reference "#PWR058") (unit 1)
         )
       )
@@
   (symbol (lib_id "Device:R") (at 127 123.19 90) (unit 1)
     (in_bom yes) (on_board yes) (dnp no)
-    (property "Reference" "R18" (at 127 118.11 90)
+    (property "Reference" "R27" (at 127 118.11 90)
       (effects (font (size 1.27 1.27)))
     )
@@
       (project "ShotClockProject"
         (path "/5fd859aa-754d-49c2-9762-3f7ebe3bb64c/1ce26b90-d7f5-4886-998a-a021d351eec6"
-          (reference "R18") (unit 1)
+          (reference "R27") (unit 1)
         )
       )
@@
   (symbol (lib_id "Switch:SW_SPST") (at 113.03 83.82 270) (unit 1)
     (in_bom yes) (on_board yes) (dnp no)
-    (property "Reference" "SW2" (at 115.57 82.55 90)
+    (property "Reference" "SW3" (at 115.57 82.55 90)
       (effects (font (size 1.27 1.27)) (justify left))
     )
@@
       (project "ShotClockProject"
         (path "/5fd859aa-754d-49c2-9762-3f7ebe3bb64c/1ce26b90-d7f5-4886-998a-a021d351eec6"
-          (reference "SW2") (unit 1)
-        )
-      )
+          (reference "SW3") (unit 1)
+        )
+      )

Commit message: Changed footprint
To horizontal 2.54 connectors
and started on rough layout
Parts:
- C4: footprint Capacitor_SMD:C_0603_1608Metric -> Capacitor_SMD:C_0402_1005Metric
- R22, R23, R24, R25, R26, R27: footprint Resistor_SMD:R_0603_1608Metric -> Resistor_SMD:R_0402_1005Metric
Changed lines of the file:
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@@
       (effects (font (size 1.27 1.27)) (justify left))
     )
-    (property "Footprint" "Capacitor_SMD:C_0603_1608Metric" (at 139.3952 88.9 0)
+    (property "Footprint" "Capacitor_SMD:C_0402_1005Metric" (at 139.3952 88.9 0)
       (effects (font (size 1.27 1.27)) hide)
     )
@@
       (effects (font (size 1.27 1.27)))
     )
-    (property "Footprint" "Resistor_SMD:R_0603_1608Metric" (at 127 102.108 90)
+    (property "Footprint" "Resistor_SMD:R_0402_1005Metric" (at 127 102.108 90)
       (effects (font (size 1.27 1.27)) hide)
     )
@@
       (effects (font (size 1.27 1.27)))
     )
-    (property "Footprint" "Resistor_SMD:R_0603_1608Metric" (at 102.87 124.968 90)
+    (property "Footprint" "Resistor_SMD:R_0402_1005Metric" (at 102.87 124.968 90)
       (effects (font (size 1.27 1.27)) hide)
     )
@@
       (effects (font (size 1.27 1.27)))
     )
-    (property "Footprint" "Resistor_SMD:R_0603_1608Metric" (at 102.87 79.248 90)
+    (property "Footprint" "Resistor_SMD:R_0402_1005Metric" (at 102.87 79.248 90)
       (effects (font (size 1.27 1.27)) hide)
     )
@@
       (effects (font (size 1.27 1.27)) (justify left))
     )
-    (property "Footprint" "Capacitor_SMD:C_0603_1608Metric" (at 139.3952 134.62 0)
+    (property "Footprint" "Capacitor_SMD:C_0402_1005Metric" (at 139.3952 134.62 0)
       (effects (font (size 1.27 1.27)) hide)
     )
@@
       (effects (font (size 1.27 1.27)))
     )
-    (property "Footprint" "Resistor_SMD:R_0603_1608Metric" (at 127 79.248 90)
+    (property "Footprint" "Resistor_SMD:R_0402_1005Metric" (at 127 79.248 90)
       (effects (font (size 1.27 1.27)) hide)
     )
@@
       (effects (font (size 1.27 1.27)))
     )
-    (property "Footprint" "Resistor_SMD:R_0603_1608Metric" (at 102.87 102.108 90)
+    (property "Footprint" "Resistor_SMD:R_0402_1005Metric" (at 102.87 102.108 90)
       (effects (font (size 1.27 1.27)) hide)
     )
@@
       (effects (font (size 1.27 1.27)) (justify left))
     )
-    (property "Footprint" "Capacitor_SMD:C_0603_1608Metric" (at 139.3952 111.76 0)
+    (property "Footprint" "Capacitor_SMD:C_0402_1005Metric" (at 139.3952 111.76 0)
       (effects (font (size 1.27 1.27)) hide)
     )
@@
       (effects (font (size 1.27 1.27)))
     )
-    (property "Footprint" "Resistor_SMD:R_0603_1608Metric" (at 127 124.968 90)
-      (effects (font (size 1.27 1.27)) hide)
-    )
+    (property "Footprint" "Resistor_SMD:R_0402_1005Metric" (at 127 124.968 90)
+      (effects (font (size 1.27 1.27)) hide)
+    )
