File: hw/ShotClockProject/STM32F103RCT6_Subsheet.kicad_sch (KiCad schematic)
At the start: 40 parts, among them J1 USB4120-03-C_REVA, J2 Conn_ST_STDC14, J3 Conn_01x06_Pin, Q1 Q_NPN_BCE, SW1 SW_SPDT, U1 STM32F103RCT6, U2 LD39015M33R, U6 USBLC6-2SC6, Y1 16MHz

Commit message: Fixed buzzer footprint
Almost done routing, 14 conn left.
Parts:
- removed BZ1: Buzzer, Buzzer_Beeper:Buzzer_CUI_CPT-9019S-SMT, symbol Device:Buzzer
- removed TP2: TestPoint, TestPoint:TestPoint_Pad_D1.0mm, symbol Connector:TestPoint
- added BUZZER1: CY-SMD-9019-3040, Cy-SMD-9019-3040:BUZ-SMD_L9.0-W9.0-P8.00-LS9.3_CY, symbol Cy-SMD-9019-3040:CY-SMD-9019-3040
Connections:
- net +3.3V: now also BUZZER1.1
- net USB_CONN_D+: no longer J1.A6 (D1+)
- net USB_CONN_D-: no longer J1.A7 (D1-)
- net at D2.2 (A), Q1.2 (C): now also BUZZER1.2
- no-connect marks 25 -> 27
Changed lines of the file:
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@@
   (junction (at 30.48 71.12) (diameter 0) (color 0 0 0 0)
   )
-  (junction (at 93.98 59.69) (diameter 0) (color 0 0 0 0)
-  )
   (junction (at 220.98 74.93) (diameter 0) (color 0 0 0 0)
   )
@@
   (junction (at 39.37 96.52) (diameter 0) (color 0 0 0 0)
   )
+  (no_connect (at 223.52 54.61))
   (no_connect (at 252.73 133.35))
   (no_connect (at 223.52 59.69))
@@
   (no_connect (at 144.78 80.01))
   (no_connect (at 144.78 128.27))
+  (no_connect (at 223.52 57.15))
   (no_connect (at 109.22 107.95))
   (no_connect (at 109.22 97.79))
@@
     (stroke (width 0) (type default))
   )
-  (wire (pts (xy 93.98 59.69) (xy 109.22 59.69))
-    (stroke (width 0) (type default))
-  )
   (wire (pts (xy 261.62 67.31) (xy 259.08 67.31))
     (stroke (width 0) (type default))
@@
     (stroke (width 0) (type default))
   )
-  (wire (pts (xy 210.82 57.15) (xy 223.52 57.15))
+  (wire (pts (xy 189.865 61.595) (xy 202.565 61.595))
     (stroke (width 0) (type default))
   )
@@
     (stroke (width 0) (type default))
   )
-  (wire (pts (xy 59.055 101.6) (xy 59.055 104.14))
+  (wire (pts (xy 59.055 101.6) (xy 59.055 105.41))
     (stroke (width 0) (type default))
   )
@@
     (stroke (width 0) (type default))
   )
-  (wire (pts (xy 59.055 109.22) (xy 59.055 110.49))
+  (wire (pts (xy 59.055 107.95) (xy 59.055 110.49))
     (stroke (width 0) (type default))
   )
@@
     (stroke (width 0) (type default))
   )
-  (wire (pts (xy 88.9 59.69) (xy 93.98 59.69))
+  (wire (pts (xy 88.9 59.69) (xy 109.22 59.69))
     (stroke (width 0) (type default))
   )
@@
     (stroke (width 0) (type default))
   )
-  (wire (pts (xy 210.82 54.61) (xy 223.52 54.61))
+  (wire (pts (xy 189.865 59.055) (xy 202.565 59.055))
     (stroke (width 0) (type default))
   )
@@
     (effects (font (size 2.5 2.5) (color 255 0 0 1)) (justify left bottom))
   )
-  (label "USB_CONN_D+" (at 210.82 54.61 0) (fields_autoplaced)
+  (label "USB_CONN_D+" (at 189.865 59.055 0) (fields_autoplaced)
     (effects (font (size 1.27 1.27)) (justify left bottom))
   )
@@
     (effects (font (size 1.27 1.27)) (justify left bottom))
   )
-  (label "USB_CONN_D-" (at 210.82 57.15 0) (fields_autoplaced)
+  (label "USB_CONN_D-" (at 189.865 61.595 0) (fields_autoplaced)
     (effects (font (size 1.27 1.27)) (justify left bottom))
   )
@@
     )
   )
+  (symbol (lib_id "Cy-SMD-9019-3040:CY-SMD-9019-3040") (at 56.515 107.95 0) (mirror y) (unit 1)
+    (in_bom yes) (on_board yes) (dnp no)
+    (property "Reference" "BUZZER1" (at 50.8 100.965 0)
+      (effects (font (size 1.27 1.27)))
+    )
+    (property "Value" "CY-SMD-9019-3040" (at 47.625 111.76 0)
+      (effects (font (size 1.27 1.27)))
+    )
+    (property "Footprint" "Cy-SMD-9019-3040:BUZ-SMD_L9.0-W9.0-P8.00-LS9.3_CY" (at 56.515 115.57 0)
+      (effects (font (size 1.27 1.27)) hide)
+    )
+    (property "Datasheet" "https://lcsc.com/product-detail/Buzzers_CY-Changzhou-Chaoyin-Elec-Cy-SMD-9019-3040_C968734.html" (at 56.515 118.11 0)
+      (effects (font (size 1.27 1.27)) hide)
+    )
+    (property "Manufacturer" "CY(超音)" (at 56.515 120.65 0)
+      (effects (font (size 1.27 1.27)) hide)
+    )
+    (property "LCSC Part" "C968734" (at 56.515 123.19 0)
+      (effects (font (size 1.27 1.27)) hide)
+    )
+    (property "JLC Part" "Extended Part" (at 56.515 125.73 0)
+      (effects (font (size 1.27 1.27)) hide)
+    )
+    (pin "1")
+    (pin "2")
+    (instances
+      (project "ShotClockProject"
+        (path "/5fd859aa-754d-49c2-9762-3f7ebe3bb64c/d53b1cd8-24cb-4dc0-9a02-0cd96c1f4291"
+          (reference "BUZZER1") (unit 1)
+        )
+      )
+    )
+  )
   (symbol (lib_id "Device:Crystal_GND24") (at 39.37 80.01 0) (unit 1)
     (in_bom yes) (on_board yes) (dnp no)
@@
     )
   )
-  (symbol (lib_id "Device:Buzzer") (at 56.515 106.68 0) (mirror y) (unit 1)
-    (in_bom yes) (on_board yes) (dnp no)
-    (property "Reference" "BZ1" (at 52.705 105.41 0)
-      (effects (font (size 1.27 1.27)) (justify left))
-    )
-    (property "Value" "Buzzer" (at 52.705 107.95 0)
-      (effects (font (size 1.27 1.27)) (justify left))
-    )
-    (property "Footprint" "Buzzer_Beeper:Buzzer_CUI_CPT-9019S-SMT" (at 57.15 104.14 90)
-      (effects (font (size 1.27 1.27)) hide)
-    )
-    (property "Datasheet" "~" (at 57.15 104.14 90)
-      (effects (font (size 1.27 1.27)) hide)
-    )
-    (pin "1")
-    (pin "2")
-    (instances
-      (project "ShotClockProject"
-        (path "/5fd859aa-754d-49c2-9762-3f7ebe3bb64c/d53b1cd8-24cb-4dc0-9a02-0cd96c1f4291"
-          (reference "BZ1") (unit 1)
-        )
-      )
-    )
-  )
   (symbol (lib_id "Device:LED") (at 85.09 82.55 0) (unit 1)
     (in_bom yes) (on_board yes) (dnp no)
@@
         )
       )
-    )
-  )
-  (symbol (lib_id "Connector:TestPoint") (at 93.98 59.69 0) (unit 1)
-    (in_bom yes) (on_board yes) (dnp no)
-    (property "Reference" "TP2" (at 95.25 55.88 0)
-      (effects (font (size 1.27 1.27)) (justify left))
-    )
-    (property "Value" "TestPoint" (at 95.25 58.42 0)
-      (effects (font (size 1.27 1.27)) (justify left))
-    )
-    (property "Footprint" "TestPoint:TestPoint_Pad_D1.0mm" (at 99.06 59.69 0)
-      (effects (font (size 1.27 1.27)) hide)
-    )
-    (property "Datasheet" "~" (at 99.06 59.69 0)
-      (effects (font (size 1.27 1.27)) hide)
-    )
-    (pin "1")
-    (instances
-      (project "ShotClockProject"
-        (path "/5fd859aa-754d-49c2-9762-3f7ebe3bb64c"
-          (reference "TP2") (unit 1)
-        )
-        (path "/5fd859aa-754d-49c2-9762-3f7ebe3bb64c/d53b1cd8-24cb-4dc0-9a02-0cd96c1f4291"
-          (reference "TP6") (unit 1)
-        )
-      )

Commit message: Added LCSC Part number
Renamed output folders
Created first output files for REV1
Parts:
- BUZZER1: LCSC Part # (none) -> C968734
- C1, C2, C3, C4, C9: LCSC Part (none) -> C1525; LCSC Part # (none) -> C1525
- C10, C11: LCSC Part (none) -> C107007; LCSC Part # (none) -> C107007
- C5: LCSC Part (none) -> C96446; LCSC Part # (none) -> C96446
- C6: LCSC Part (none) -> C15195; LCSC Part # (none) -> C15195
- C7, C8, C9: LCSC Part (none) -> C52923; LCSC Part # (none) -> C52923
- D1: LCSC Part (none) -> C264451; LCSC Part # (none) -> C264451
- D2: LCSC Part (none) -> C2128; LCSC Part # (none) -> C2128
- FB1: LCSC Part (none) -> C127301; LCSC Part # (none) -> C127301
- J1: LCSC Part (none) -> C5187468; LCSC Part # (none) -> C5187468
- J2: LCSC Part (none) -> C3975190; LCSC Part # (none) -> C3975190
- J3: LCSC Part (none) -> C56816; LCSC Part # (none) -> C56816
- Q1: LCSC Part (none) -> C111113; LCSC Part # (none) -> C111113
- R1: LCSC Part (none) -> C25744; LCSC Part # (none) -> C25744
- R2: LCSC Part (none) -> C25076; LCSC Part # (none) -> C25076
- R2: LCSC Part (none) -> C105637; LCSC Part # (none) -> C105637
- R2: LCSC Part (none) -> C477610; LCSC Part # (none) -> C477610
- R2: LCSC Part (none) -> C25102; LCSC Part # (none) -> C25102
- R2: LCSC Part (none) -> C25867; LCSC Part # (none) -> C25867
- R2: LCSC Part (none) -> C25905; LCSC Part # (none) -> C25905
- SW1: LCSC Part (none) -> C500057; LCSC Part # (none) -> C500057
- U1: LCSC Part (none) -> C8323; LCSC Part # (none) -> C8323
- U2: LCSC Part (none) -> C2798212; LCSC Part # (none) -> C2798212
- U6: LCSC Part (none) -> C7519; LCSC Part # (none) -> C7519
- Y1: LCSC Part (none) -> C112972; LCSC Part # (none) -> C112972
