File: hw/ShotClockProject/Regulator5V.kicad_sch (KiCad schematic)
At the start: 12 parts, among them U2 TPS63000

Commit message: Finished routing and added silk + part nmbr
Parts:
- C14: LCSC Part # C1525 -> (none)
- C15, C16, C17: LCSC Part # C96446 -> (none)
- C18: LCSC Part # C1559 -> (none)
- D2: LCSC Part # C72043 -> (none)
- L1: LCSC Part # C404494 -> (none)
- R10: LCSC Part # C25076 -> (none)
- R10: LCSC Part # C25867 -> (none)
- R11: LCSC Part # C144787 -> (none)
- R12: LCSC Part # C25745 -> (none)
- U2: LCSC Part # C24966 -> (none)
Changed lines of the file:
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@@
       (effects (font (size 1.27 1.27)) hide)
     )
-    (property "LCSC Part #" "C24966" (at 86.36 48.26 0)
+    (property "LCSC Part #" "" (at 86.36 48.26 0)
       (effects (font (size 1.27 1.27)) hide)
     )
@@
       (effects (font (size 1.27 1.27)) hide)
     )
-    (property "LCSC Part #" "C96446" (at 48.26 52.07 0)
+    (property "LCSC Part #" "" (at 48.26 52.07 0)
       (effects (font (size 1.27 1.27)) hide)
     )
@@
       (effects (font (size 1.27 1.27)) hide)
     )
-    (property "LCSC Part #" "C72043" (at 154.94 45.72 0)
+    (property "LCSC Part #" "" (at 154.94 45.72 0)
       (effects (font (size 1.27 1.27)) hide)
     )
@@
       (effects (font (size 1.27 1.27)) hide)
     )
-    (property "LCSC Part #" "C96446" (at 144.78 44.45 0)
+    (property "LCSC Part #" "" (at 144.78 44.45 0)
       (effects (font (size 1.27 1.27)) hide)
     )
@@
       (effects (font (size 1.27 1.27)) hide)
     )
-    (property "LCSC Part #" "C25076" (at 59.69 41.91 0)
+    (property "LCSC Part #" "" (at 59.69 41.91 0)
       (effects (font (size 1.27 1.27)) hide)
     )
@@
       (effects (font (size 1.27 1.27)) hide)
     )
-    (property "LCSC Part #" "C96446" (at 134.62 44.45 0)
+    (property "LCSC Part #" "" (at 134.62 44.45 0)
       (effects (font (size 1.27 1.27)) hide)
     )
@@
       (effects (font (size 1.27 1.27)) hide)
     )
-    (property "LCSC Part #" "C25867" (at 154.94 54.61 0)
+    (property "LCSC Part #" "" (at 154.94 54.61 0)
       (effects (font (size 1.27 1.27)) hide)
     )
@@
       (effects (font (size 1.27 1.27)) hide)
     )
-    (property "LCSC Part #" "C1525" (at 59.69 52.07 0)
+    (property "LCSC Part #" "" (at 59.69 52.07 0)
       (effects (font (size 1.27 1.27)) hide)
     )
@@
       (effects (font (size 1.27 1.27)) hide)
     )
-    (property "LCSC Part #" "C25745" (at 102.87 49.53 0)
+    (property "LCSC Part #" "" (at 102.87 49.53 0)
       (effects (font (size 1.27 1.27)) hide)
     )
@@
       (effects (font (size 1.27 1.27)) hide)
     )
-    (property "LCSC Part #" "C1559" (at 113.03 41.91 0)
+    (property "LCSC Part #" "" (at 113.03 41.91 0)
       (effects (font (size 1.27 1.27)) hide)
     )
@@
       (effects (font (size 1.27 1.27)) hide)
     )
-    (property "LCSC Part #" "C404494" (at 73.66 53.34 0)
+    (property "LCSC Part #" "" (at 73.66 53.34 0)
       (effects (font (size 1.27 1.27)) hide)
     )
@@
       (effects (font (size 1.27 1.27)) hide)
     )
-    (property "LCSC Part #" "C144787" (at 102.87 41.91 0)
-      (effects (font (size 1.27 1.27)) hide)
-    )
+    (property "LCSC Part #" "" (at 102.87 41.91 0)
+      (effects (font (size 1.27 1.27)) hide)
+    )
