File: hw/ShotClockProject/Regulator5V.kicad_sch (KiCad schematic)
At the start: 12 parts, among them U2 TPS63000

Commit message: Add REV3 odt file, update CubeMX version and fix the ADC readout for battery voltage.
Parts:
- renumbered C18 to C22, C17 to C23, C16 to C24, C15 to C25, C14 to C26, D2 to D5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
