File: hw/ShotClockProject/Regulator3V3.kicad_sch (KiCad schematic)
At the start: 12 parts, among them U2 TPS63000

Commit message: Add REV3 odt file, update CubeMX version and fix the ADC readout for battery voltage.
Parts:
- renumbered C18 to C17, C17 to C18, C16 to C19, C15 to C20, C14 to C21, D2 to D4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
