File: hw/ShotClockProject/buzzer_3v3_pwm.kicad_sch (KiCad schematic)
At the start: 5 parts, among them Q1 Q_NPN_BCE

Commit message: Added I2C support
Calculated pull-up resistor values
Added 6 pin female headers to mainboard
Added nRESET line for the I2C chips
Removed PCB routing and part placement
Parts:
- renumbered D2 to D6, Q1 to Q4
Changed lines of the file:
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@@
   (symbol (lib_id "Diode:1N4148") (at 144.78 95.885 90) (mirror x) (unit 1)
     (in_bom yes) (on_board yes) (dnp no) (fields_autoplaced)
-    (property "Reference" "D2" (at 142.24 94.615 90)
+    (property "Reference" "D6" (at 142.24 94.615 90)
       (effects (font (size 1.27 1.27)) (justify left))
     )
@@
       (project "ShotClockProject"
         (path "/5fd859aa-754d-49c2-9762-3f7ebe3bb64c/0090141d-207a-4f3a-bfd6-43ff1a882302"
-          (reference "D2") (unit 1)
+          (reference "D6") (unit 1)
         )
       )
@@
         )
         (path "/5fd859aa-754d-49c2-9762-3f7ebe3bb64c/0090141d-207a-4f3a-bfd6-43ff1a882302"
-          (reference "R11") (unit 1)
+          (reference "R35") (unit 1)
         )
       )
@@
         )
         (path "/5fd859aa-754d-49c2-9762-3f7ebe3bb64c/0090141d-207a-4f3a-bfd6-43ff1a882302"
-          (reference "#PWR023") (unit 1)
+          (reference "#PWR085") (unit 1)
         )
       )
@@
         )
         (path "/5fd859aa-754d-49c2-9762-3f7ebe3bb64c/0090141d-207a-4f3a-bfd6-43ff1a882302"
-          (reference "R10") (unit 1)
+          (reference "R34") (unit 1)
         )
       )
@@
         )
         (path "/5fd859aa-754d-49c2-9762-3f7ebe3bb64c/0090141d-207a-4f3a-bfd6-43ff1a882302"
-          (reference "#PWR018") (unit 1)
+          (reference "#PWR084") (unit 1)
         )
       )
@@
   (symbol (lib_id "Device:Q_NPN_BCE") (at 147.32 106.045 0) (unit 1)
     (in_bom yes) (on_board yes) (dnp no)
-    (property "Reference" "Q1" (at 152.4 104.775 0)
+    (property "Reference" "Q4" (at 152.4 104.775 0)
       (effects (font (size 1.27 1.27)) (justify left))
     )
@@
       (project "ShotClockProject"
         (path "/5fd859aa-754d-49c2-9762-3f7ebe3bb64c/0090141d-207a-4f3a-bfd6-43ff1a882302"
-          (reference "Q1") (unit 1)
+          (reference "Q4") (unit 1)
         )
       )
@@
         )
         (path "/5fd859aa-754d-49c2-9762-3f7ebe3bb64c/0090141d-207a-4f3a-bfd6-43ff1a882302"
-          (reference "#PWR022") (unit 1)
-        )
-      )
+          (reference "#PWR086") (unit 1)
+        )
+      )

Commit message: Finished mainboard routing
Reconfigered pins to make routing easier/cleaner
Placed copper fills as much as possible to create an even plating index
Connections:
- net buzz2: now reaches BUZZER1.2, D6.2 (A), Q4.2 (C)
Other:
- moved on the sheet: BUZZER1
Changed lines of the file:
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@@
   (junction (at 149.86 90.805) (diameter 0) (color 0 0 0 0)
   )
+  (wire (pts (xy 161.925 90.805) (xy 149.86 90.805))
+    (stroke (width 0) (type default))
+  )
   (wire (pts (xy 140.97 106.045) (xy 138.43 106.045))
+    (stroke (width 0) (type default))
+  )
+  (wire (pts (xy 161.925 99.695) (xy 149.86 99.695))
     (stroke (width 0) (type default))
   )
@@
     (stroke (width 0) (type default))
   )
-  (wire (pts (xy 149.86 90.805) (xy 149.86 94.615))
+  (wire (pts (xy 161.925 90.805) (xy 161.925 94.615))
     (stroke (width 0) (type default))
   )
-  (wire (pts (xy 149.86 97.155) (xy 149.86 99.695))
+  (wire (pts (xy 161.925 97.155) (xy 161.925 99.695))
     (stroke (width 0) (type default))
   )
@@
   (wire (pts (xy 149.86 89.535) (xy 149.86 90.805))
     (stroke (width 0) (type default))
+  )
+  (label "buzz2" (at 153.67 99.695 0) (fields_autoplaced)
+    (effects (font (size 1.27 1.27)) (justify left bottom))
   )
   (hierarchical_label "buzzer_pwm_in" (shape input) (at 129.54 106.045 180) (fields_autoplaced)
@@
     )
   )
-  (symbol (lib_id "Cy-SMD-9019-3040:CY-SMD-9019-3040") (at 152.4 97.155 0) (unit 1)
+  (symbol (lib_id "Cy-SMD-9019-3040:CY-SMD-9019-3040") (at 164.465 97.155 0) (unit 1)
     (in_bom yes) (on_board yes) (dnp no)
-    (property "Reference" "BUZZER1" (at 158.115 90.17 0)
+    (property "Reference" "BUZZER1" (at 170.18 90.17 0)
       (effects (font (size 1.27 1.27)))
     )
-    (property "Value" "CY-SMD-9019-3040" (at 161.29 100.965 0)
+    (property "Value" "CY-SMD-9019-3040" (at 173.355 100.965 0)
       (effects (font (size 1.27 1.27)))
     )
-    (property "Footprint" "Cy-SMD-9019-3040:BUZ-SMD_L9.0-W9.0-P8.00-LS9.3_CY" (at 152.4 104.775 0)
+    (property "Footprint" "Cy-SMD-9019-3040:BUZ-SMD_L9.0-W9.0-P8.00-LS9.3_CY" (at 164.465 104.775 0)
       (effects (font (size 1.27 1.27)) hide)
     )
-    (property "Datasheet" "https://lcsc.com/product-detail/Buzzers_CY-Changzhou-Chaoyin-Elec-Cy-SMD-9019-3040_C968734.html" (at 152.4 107.315 0)
+    (property "Datasheet" "https://lcsc.com/product-detail/Buzzers_CY-Changzhou-Chaoyin-Elec-Cy-SMD-9019-3040_C968734.html" (at 164.465 107.315 0)
       (effects (font (size 1.27 1.27)) hide)
     )
-    (property "Manufacturer" "CY(超音)" (at 152.4 109.855 0)
+    (property "Manufacturer" "CY(超音)" (at 164.465 109.855 0)
       (effects (font (size 1.27 1.27)) hide)
     )
-    (property "JLC Part" "Extended Part" (at 152.4 114.935 0)
+    (property "JLC Part" "Extended Part" (at 164.465 114.935 0)
       (effects (font (size 1.27 1.27)) hide)
     )
-    (property "LCSC Part #" "C968734" (at 152.4 97.155 0)
+    (property "LCSC Part #" "C968734" (at 164.465 97.155 0)
       (effects (font (size 1.27 1.27)) hide)
     )
-    (property "LCSC Part" "C968734" (at 152.4 97.155 0)
+    (property "LCSC Part" "C968734" (at 164.465 97.155 0)
       (effects (font (size 1.27 1.27)) hide)
     )

Commit message: Finished routing and added silk + part nmbr
Parts:
- BUZZER1: LCSC Part # C968734 -> (none)
- D6: LCSC Part # C2128 -> (none)
- Q4: LCSC Part # C111113 -> (none)
- R2: LCSC Part # C105637 -> (none)
- R2: LCSC Part # C25102 -> (none)
Changed lines of the file:
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@@
       (effects (font (size 1.27 1.27)) hide)
     )
-    (property "LCSC Part #" "C2128" (at 144.78 95.885 0)
+    (property "LCSC Part #" "" (at 144.78 95.885 0)
       (effects (font (size 1.27 1.27)) hide)
     )
@@
       (effects (font (size 1.27 1.27)) hide)
     )
-    (property "LCSC Part #" "C968734" (at 164.465 97.155 0)
+    (property "LCSC Part #" "" (at 164.465 97.155 0)
       (effects (font (size 1.27 1.27)) hide)
     )
@@
       (effects (font (size 1.27 1.27)) hide)
     )
-    (property "LCSC Part #" "C105637" (at 140.97 109.855 0)
+    (property "LCSC Part #" "" (at 140.97 109.855 0)
       (effects (font (size 1.27 1.27)) hide)
     )
@@
       (effects (font (size 1.27 1.27)) hide)
     )
-    (property "LCSC Part #" "C25102" (at 134.62 106.045 0)
+    (property "LCSC Part #" "" (at 134.62 106.045 0)
       (effects (font (size 1.27 1.27)) hide)
     )
@@
       (effects (font (size 1.27 1.27)) hide)
     )
-    (property "LCSC Part #" "C111113" (at 147.32 106.045 0)
+    (property "LCSC Part #" "" (at 147.32 106.045 0)
       (effects (font (size 1.27 1.27)) hide)
     )

Commit message: Add REV3 odt file, update CubeMX version and fix the ADC readout for battery voltage.
Parts:
- renumbered R2 to R34, R2 to R35
